File: schematic/v3/APM.kicad_sch (KiCad schematic)
At the start: 13 parts, among them J12 AUDIO_OUT, J4 LCD_display, U1 NUCLEO-H753ZI

Commit message: progress on creating APM board first
Other:
- note added: "Audio Peripheral Module"
Changed lines of the file:
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@@
 		(rev "2")
+	)
+	(text "Audio Peripheral Module"
+		(exclude_from_sim no)
+		(at 32.258 24.13 0)
+		(effects
+			(font
+				(size 1.905 1.905)
+			)
+		)
 	)
 	(text "STM32H755 NUCLEO"
