File: schematic/v3/TDM_pwr_mon.kicad_sch (KiCad schematic)
At the start: 42 parts, among them J10 INA219_CONFIG, J11 INA219_CONFIG, J15 INA219_CONFIG, J5 INA219_CONFIG, J6 INA219_CONFIG, J7 INA219_CONFIG, U10 INA219AxD, U11 INA219AxD, U12 INA219AxD, U13 INA219AxD, U20 INA219AxD, U7 INA219AxD

Commit message: progress on creating APM board first
Connections:
- net at J15.1 (Pin_1), R4.2, U20.1 (A1): no longer J15.2 (Pin_2), R3.2, U20.2 (A0)
- net at J6.1 (Pin_1), R21.2, U10.1 (A1): no longer J6.2 (Pin_2), R20.2, U10.2 (A0)
- net at J5.1 (Pin_1), R14.2, U7.1 (A1): no longer J5.2 (Pin_2), R13.2, U7.2 (A0)
- net at J10.1 (Pin_1), R25.2, U12.1 (A1): no longer J10.2 (Pin_2), R23.2, U12.2 (A0)
- net at J11.1 (Pin_1), R28.2, U13.1 (A1): no longer J11.2 (Pin_2), R26.2, U13.2 (A0)
- net at J7.1 (Pin_1), R24.2, U11.1 (A1): no longer J7.2 (Pin_2), R22.2, U11.2 (A0)
- new net: J15.2 (Pin_2), R3.2, U20.2 (A0)
- new net: J6.2 (Pin_2), R20.2, U10.2 (A0)
- new net: J5.2 (Pin_2), R13.2, U7.2 (A0)
- new net: J10.2 (Pin_2), R23.2, U12.2 (A0)
- new net: J11.2 (Pin_2), R26.2, U13.2 (A0)
- new net: J7.2 (Pin_2), R22.2, U11.2 (A0)
Changed lines of the file:
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@@
-	)
-	(junction
-		(at 132.08 96.52)
-		(diameter 0)
-		(color 0 0 0 0)
 	)
 	(junction
@@
 	)
 	(junction
-		(at 186.69 137.16)
-		(diameter 0)
-		(color 0 0 0 0)
-	)
-	(junction
 		(at 167.64 38.1)
 		(diameter 0)
@@
 	)
 	(junction
-		(at 132.08 55.88)
-		(diameter 0)
-		(color 0 0 0 0)
-	)
-	(junction
 		(at 179.07 96.52)
 		(diameter 0)
@@
 	)
 	(junction
-		(at 186.69 96.52)
-		(diameter 0)
-		(color 0 0 0 0)
-	)
-	(junction
 		(at 179.07 137.16)
 		(diameter 0)
@@
 	)
 	(junction
-		(at 132.08 137.16)
-		(diameter 0)
-		(color 0 0 0 0)
-	)
-	(junction
 		(at 113.03 78.74)
 		(diameter 0)
@@
 	)
 	(junction
-		(at 186.69 55.88)
-		(diameter 0)
-		(color 0 0 0 0)
-	)
-	(junction
 		(at 102.87 53.34)
 		(diameter 0)
@@
 	(wire
 		(pts
-			(xy 132.08 55.88) (xy 135.89 55.88)
+			(xy 124.46 55.88) (xy 135.89 55.88)
 		)
 		(stroke
@@
 	(wire
 		(pts
-			(xy 132.08 96.52) (xy 135.89 96.52)
+			(xy 124.46 96.52) (xy 135.89 96.52)
 		)
 		(stroke
@@
 	(wire
 		(pts
-			(xy 179.07 96.52) (xy 186.69 96.52)
+			(xy 179.07 96.52) (xy 190.5 96.52)
 		)
 		(stroke
@@
 	(wire
 		(pts
-			(xy 124.46 137.16) (xy 132.08 137.16)
-		)
-		(stroke
-			(width 0)
-			(type default)
-		)
-	)
-	(wire
-		(pts
 			(xy 101.6 119.38) (xy 104.14 119.38)
 		)
@@
 	(wire
 		(pts
-			(xy 124.46 96.52) (xy 132.08 96.52)
-		)
-		(stroke
-			(width 0)
-			(type default)
-		)
-	)
-	(wire
-		(pts
-			(xy 124.46 55.88) (xy 132.08 55.88)
-		)
-		(stroke
-			(width 0)
-			(type default)
-		)
-	)
-	(wire
-		(pts
 			(xy 146.05 100.33) (xy 147.32 100.33)
 		)
@@
 	(wire
 		(pts
-			(xy 179.07 137.16) (xy 186.69 137.16)
+			(xy 179.07 137.16) (xy 190.5 137.16)
 		)
 		(stroke
@@
 	(wire
 		(pts
-			(xy 132.08 137.16) (xy 135.89 137.16)
+			(xy 124.46 137.16) (xy 135.89 137.16)
 		)
 		(stroke
@@
 	(wire
 		(pts
-			(xy 186.69 55.88) (xy 190.5 55.88)
+			(xy 179.07 55.88) (xy 190.5 55.88)
 		)
 		(stroke
@@
 	(wire
 		(pts
-			(xy 186.69 96.52) (xy 190.5 96.52)
-		)
-		(stroke
-			(width 0)
-			(type default)
-		)
-	)
-	(wire
-		(pts
-			(xy 179.07 55.88) (xy 186.69 55.88)
-		)
-		(stroke
-			(width 0)
-			(type default)
-		)
-	)
-	(wire
-		(pts
 			(xy 132.08 53.34) (xy 135.89 53.34)
 		)
@@
 		)
 		(stroke
-			(width 0)
-			(type default)
-		)
-	)
-	(wire
-		(pts
-			(xy 186.69 137.16) (xy 190.5 137.16)
-		)
-		(stroke
