File: schematic/v4/APM/PMS_APM.kicad_sch (KiCad schematic)
At the start: 7 parts, among them J11 INA219_CONFIG, U13 INA219AxD

Commit message: progress on board sep
Other:
- note added: "PMS has an INA219 current sensor for each board/node in the PCB. Each takes in the 5V from it's parent board and supplies 5V to said board's circuit (its peripherals) thus enabling monitoring"
- note removed: "PMS has an INA219 current sensor for each board/node in on the PCB. Each takes in the 5V from it's parent board and supplies 5V to said board's circuit (its peripherals) thus enabling monitoring"
Changed lines of the file:
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@@
 		)
 	)
-	(text "PMS has an INA219 current sensor\nfor each board/node in on the \nPCB. Each takes in the 5V from it's\nparent board and supplies 5V to said\nboard's circuit (its peripherals)\nthus enabling monitoring"
+	(text "PMS has an INA219 current sensor\nfor each board/node in the \nPCB. Each takes in the 5V from it's\nparent board and supplies 5V to said\nboard's circuit (its peripherals)\nthus enabling monitoring"
 		(exclude_from_sim no)
 		(at 34.29 30.734 0)
@@
 	)
 	(junction
-		(at 121.92 87.63)
-		(diameter 0)
-		(color 0 0 0 0)
-	)
-	(junction
 		(at 149.86 95.25)
 		(diameter 0)
@@
 	(wire
 		(pts
-			(xy 121.92 87.63) (xy 128.27 87.63)
-		)
-		(stroke
-			(width 0)
-			(type default)
-		)
-	)
-	(wire
-		(pts
 			(xy 151.13 87.63) (xy 148.59 87.63)
 		)
@@
 	(wire
 		(pts
-			(xy 119.38 87.63) (xy 121.92 87.63)
+			(xy 119.38 87.63) (xy 128.27 87.63)
 		)
 		(stroke
@@
 					(unit 1)
 				)
-			)
-		)
-	)
-	(symbol
-		(lib_id "power:PWR_FLAG")
-		(at 121.92 87.63 0)
-		(unit 1)
-		(exclude_from_sim no)
-		(in_bom yes)
-		(on_board yes)
-		(dnp no)
-		(fields_autoplaced yes)
-		(property "Reference" "#FLG012"
-			(at 121.92 85.725 0)
-			(effects
-				(font
-					(size 1.27 1.27)
-				)
-				(hide yes)
-			)
-		)
-		(property "Value" "PWR_FLAG"
-			(at 121.92 82.55 0)
-			(effects
-				(font
-					(size 1.27 1.27)
-				)
-			)
-		)
-		(property "Footprint" ""
-			(at 121.92 87.63 0)
-			(effects
-				(font
-					(size 1.27 1.27)
-				)
-				(hide yes)
-			)
-		)
-		(property "Datasheet" "~"
-			(at 121.92 87.63 0)
-			(effects
-				(font
-					(size 1.27 1.27)
-				)
-				(hide yes)
-			)
-		)
-		(property "Description" "Special symbol for telling ERC where power comes from"
-			(at 121.92 87.63 0)
-			(effects
-				(font
-					(size 1.27 1.27)
-				)
-				(hide yes)
-			)
-		)
-		(pin "1"
-		)
-		(instances
-			(project "APM"
-				(path "/63e257c1-2fa4-4533-ab9e-932d24befb8c/4ce745b1-4412-4127-8e92-31b01ddd3f60"
-					(reference "#FLG012")
-					(unit 1)
-				)

Commit message: should be good for refab and actual layout. may need better BOM matching tho
Parts:
- J11: footprint Connector_PinHeader_1.27mm:PinHeader_1x02_P1.27mm_Vertical -> Connector_PinHeader_2.54mm:PinHeader_1x02_P2.54mm_Vertical
Changed lines of the file:
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@@
 			)
 		)
-		(property "Footprint" "Connector_PinHeader_1.27mm:PinHeader_1x02_P1.27mm_Vertical"
+		(property "Footprint" "Connector_PinHeader_2.54mm:PinHeader_1x02_P2.54mm_Vertical"
 			(at 166.37 92.71 0)
 			(effects
