File: schematic/v5/APM/APM.kicad_pcb (KiCad board)
At the start: 4 copper layers, 72.5 x 104.5 mm, 77 parts, among them J1 ACM_CTRL, J11 INA219_CONFIG, J12 AUDIO_OUT, J13 Conn_02x36_Odd_Even, J14 periperhals, J15 Conn_02x36_Odd_Even, J2 CAN, J21 USB_A, J29 USB_A, J3 7SDD_CTRL, J30 UART_DEBUG, J4 LCD_display, J5 INTRPT, J7 TDM_PMS_I2C, SW1 WARN_RST, SW2 FAIL_RST, U1 NUCLEO-H753ZI, U13 INA219AxD, U38 CH340G, Y7 12MHz

Commit message: starting 7sdd board
Other:
- board text added: "signalmesh APM dev board v2 rev3 Akiel Aries"
- board text removed: "signalmesh APM dev board v2 rev4 Akiel Aries"
Changed lines of the file:
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@@
 		)
 	)
-	(gr_text "signalmesh APM dev board \nv2 rev4\nAkiel Aries"
+	(gr_text "signalmesh APM dev board \nv2 rev3\nAkiel Aries"
 		(at 114.05 155.075 0)
 		(layer "B.SilkS")
