File: schematic/v5/APM/7SDD/7SDD.kicad_pcb (KiCad board)
At the start: 2 copper layers, 37 parts, among them J2 Conn_01x04_Pin, J3 USB_B_Micro, J4 STLINK, SW1 SW_SPDT, U1 AMS1117-3.3, U2 STM32F103C8T6, U3 HDSP-7501, U4 HDSP-7501, U5 HDSP-7501, U7 HDSP-7501, Y1 16 MHz

Commit message: hmmm
Parts:
- moved H1 11.8 mm to (177.8, 87.6)
- moved H2 11.8 mm to (220.6, 87.5)
- moved J3 2.66 mm to (212.4, 95.7)
- moved J2 1.00 mm to (206.6, 88.3)
Routing:
- net /STM32F103/SEG_E: track 10.3 -> 31.2 mm
- net /STM32F103/SEG_D: track 10.3 -> 31.2 mm
- net /STM32F103/SEG_F: track 10.3 -> 31.1 mm
- net /STM32F103/SEG_B: track 10.4 -> 31.1 mm
- net /STM32F103/SEG_G: track 10.3 -> 31.1 mm
- net /STM32F103/SEG_DP: track 10.4 -> 31.1 mm
- net /STM32F103/SEG_A: track 10.4 -> 31.1 mm
- net /STM32F103/SEG_C: track 10.4 -> 31.0 mm
- net Net-(R3-Pad2): track 0.00 -> 3.43 mm
- net Net-(R6-Pad2): track 0.00 -> 3.42 mm
- net Net-(R7-Pad2): track 0.00 -> 3.38 mm
- net Net-(R2-Pad2): track 0.00 -> 3.37 mm
