File: schematic/APM_v3_r1/APM.kicad_pcb (KiCad board)
At the start: 4 copper layers, 72.5 x 104.5 mm, 97 parts, among them J1 ACM_CTRL, J11 DAC_L_PRB, J12 Conn_01x02, J13 Conn_02x36_Odd_Even, J14 ADC FFC, J15 FPGA FFC, J16 USB_A, J17 MIDI_DGB, J18 Conn_02x36_Odd_Even, J2 CAN, J29 USB_A, J3 7SDD_CTRL, J30 UART_DEBUG, J4 LCD_display, J5 INTRPT, J7 DAC_R_PRB, U1 NUCLEO-H753ZI, U13 INA219AxD, U2 CH340G, U3 LT1963AxST-3.3, U38 CH340G, U4 W25Q128JVS, U5 MR25H40, U7 INA219AxD, U8 24LC1025-I_P, Y1 12MHz, Y7 12MHz

Commit message: ground planes on f and b cu
Parts:
- added J19: FPGA_QSPI, Connector_PinHeader_2.54mm:PinHeader_1x06_P2.54mm_Vertical, B.Cu at (98.9, 136.7)
- added J20: FPGA_UART, Connector_PinHeader_2.54mm:PinHeader_1x02_P2.54mm_Vertical, B.Cu at (105.7, 136.7)
- added J21: APM_FPGA_UART, Connector_PinHeader_2.54mm:PinHeader_1x02_P2.54mm_Vertical, B.Cu at (105.7, 132.1)
- added J22: FPGA_SPI, Connector_PinHeader_2.54mm:PinHeader_1x04_P2.54mm_Vertical, B.Cu at (86.3, 131.2)
- U8: moved to B.Cu
- moved G*** 17.2 mm to (83.5, 120.0)
- moved REF** 15.3 mm to (72.5, 150.9)
- moved R30 10.5 mm to (80.0, 92.4)
- moved D7 10.5 mm to (80.0, 89.9)
- moved J5 8.96 mm to (121.3, 146.5)
- moved R18 7.65 mm to (106.3, 111.8)
- moved JP5 7.65 mm to (104.5, 112.1)
- moved JP3 7.03 mm to (111.8, 112.1)
- moved R8 7.03 mm to (113.7, 111.8)
- moved J3 6.88 mm to (121.3, 134.5)
- moved REF** 5.56 mm to (114.8, 143.1)
- moved TH5 4.11 mm to (95.8, 123.3)
- moved TP3 4.11 mm to (98.5, 123.1)
- moved R9 4.11 mm to (94.7, 120.2)
- moved D19 2.60 mm to (97.2, 140.3)
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Connections:
- J13 pad 29: /ADC_1-16_POT_1 -> unconnected-(J13-Pin_29-Pad29)
- J13 pad 33: /ADC_1-5_POT_2 -> /SPIFLASH_CS
- J13 pad 35: /ADC_1-10_POT_3 -> /SPIMRAM_CS
- J13 pad 36: /ADC_3-1_POT_4 -> unconnected-(J13-Pin_36-Pad36)
- J13 pad 37: unconnected-(J13-Pin_37-Pad37) -> /APM_MRAM_EN
- J13 pad 39: unconnected-(J13-Pin_39-Pad39) -> /APM_SPIFLASH_EN
- J13 pad 42: unconnected-(J13-Pin_42-Pad42) -> /APM_EEPROM_EN
- J13 pad 51: /SPIFLASH_CS -> unconnected-(J13-Pin_51-Pad51)
- J13 pad 53: /SPIMRAM_CS -> unconnected-(J13-Pin_53-Pad53)
- J13 pad 55: /SPIFPGA_CS -> unconnected-(J13-Pin_55-Pad55)
- J13 pad 59: unconnected-(J13-Pin_59-Pad59) -> /SPIFPGA_CS
- J13 pad 64: /APM_SPIFLASH_EN -> unconnected-(J13-Pin_64-Pad64)
- J13 pad 66: /APM_MRAM_EN -> unconnected-(J13-Pin_66-Pad66)
- J13 pad 68: /APM_EEPROM_EN -> unconnected-(J13-Pin_68-Pad68)
- J15 pad 35: unconnected-(J15-Pin_35-Pad35) -> /FPGA_UART_TX
- J15 pad 37: unconnected-(J15-Pin_37-Pad37) -> /FPGA_UART_RX
- U4 pad 2: /APM_SPI1_MISO -> /APM_SPI4_MISO
- U4 pad 5: /APM_SPI1_MOSI -> /APM_SPI4_MOSI
- U4 pad 6: /APM_SPI1_SCK -> /APM_SPI4_SCK
- U5 pad 2: /APM_SPI1_MISO -> /APM_SPI4_MISO
- U5 pad 5: /APM_SPI1_MOSI -> /APM_SPI4_MOSI
- U5 pad 6: /APM_SPI1_SCK -> /APM_SPI4_SCK
Routing:
- net /APM_SPI4_MOSI: track 0.00 -> 71.5 mm, vias 0 -> 2
- net /APM_SPI1_CLK: track 0.00 -> 42.4 mm
- net /APM_SPI4_MISO: track 0.00 -> 42.2 mm, vias 0 -> 3
- net /APM_SPI4_SCK: track 0.00 -> 40.7 mm, vias 0 -> 4
- net /APM_SPI1_MISO: track 0.00 -> 40.0 mm
- net /APM_SPI1_MOSI: track 0.00 -> 36.5 mm
- net /APM_SPI1_CS: track 0.00 -> 32.9 mm
- net /APM_MRAM_EN: track 58.7 -> 27.3 mm
- net /APM_SPIFLASH_EN: track 45.2 -> 18.4 mm, vias 3 -> 1
- net /SPIMRAM_CS: track 47.7 -> 25.0 mm
- net /SPIFLASH_CS: track 38.0 -> 16.2 mm, vias 1 -> 0
- net /APM_FPGA_UART_TX: track 0.00 -> 18.8 mm
- net /APM_EEPROM_EN: track 41.1 -> 23.0 mm
- net /APM_FPGA_UART_RX: track 0.00 -> 17.6 mm, vias 0 -> 2
- net /FPGA_UART_TX: track 0.00 -> 17.1 mm, vias 0 -> 2
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- added copper zone on F.Cu, net GND
- removed copper zone on B.Cu, net /THRM_C
Other:
- board text added: "CLK"
- board text added: "CS"
- board text added: "IO0"
- board text added: "IO1"
- board text added: "IO2"
- board text added: "IO3"
- board text added: "MISO"
- board text added: "MOSI"
- board text added: "NCS"

Commit message: getting APM V3 R1 made. starting R2
Parts:
- removed J22: FPGA_SPI, Connector_PinHeader_2.54mm:PinHeader_1x04_P2.54mm_Vertical
- added C8: 100nF, Capacitor_SMD:C_0805_2012Metric, B.Cu at (78.7, 115.3)
- added CLK1: ~, TestPoint:TestPoint_Pad_D1.0mm, B.Cu at (112.5, 127.2)
- added CS1: ~, TestPoint:TestPoint_Pad_D1.0mm, B.Cu at (101.8, 127.2)
- added J23: QSPIFLASH, Connector_PinHeader_2.54mm:PinHeader_1x06_P2.54mm_Vertical, B.Cu at (98.9, 131.4)
- added MISO1: ~, TestPoint:TestPoint_Pad_D1.0mm, B.Cu at (109.0, 127.2)
- added MOSI1: ~, TestPoint:TestPoint_Pad_D1.0mm, B.Cu at (105.4, 127.2)
- added U6: W25Q128JVS, Package_SO:SOIC-8_5.3x5.3mm_P1.27mm, B.Cu at (81.7, 119.5)
- moved G*** 46.2 mm to (109.8, 81.9)
- moved TH5 3.56 mm to (95.0, 119.9)
- moved TP3 3.31 mm to (99.5, 120.0)
- moved R9 2.66 mm to (97.3, 120.0)
- moved R42 1.77 mm to (98.9, 141.1), turned to 0 degrees
Routing:
- net /STORAGE_APM/QSPIFLASH_CS: track 0.00 -> 20.4 mm
- net /APM_SPI1_CLK: track 42.4 -> 22.1 mm
- net /STORAGE_APM/QSPIFLASH_IO3: track 0.00 -> 19.4 mm
- net /APM_SPI1_MISO: track 40.0 -> 21.2 mm
- net /STORAGE_APM/QSPIFLASH_IO1: track 0.00 -> 18.0 mm
- net /STORAGE_APM/QSPIFLASH_CLK: track 0.00 -> 17.2 mm
- net 3V3_APM: track 100.3 -> 116.2 mm, vias 5 -> 6
- net /APM_I2C1_SDA: track 0.00 -> 15.7 mm, vias 0 -> 2
- net /STORAGE_APM/QSPIFLASH_IO2: track 0.00 -> 15.6 mm
- net /APM_I2C1_SCL: track 0.00 -> 15.4 mm, vias 0 -> 2
- net /STORAGE_APM/QSPIFLASH_IO0: track 0.00 -> 14.6 mm
- net /APM_SPI1_MOSI: track 36.5 -> 22.5 mm
- net 3V3_LDO: track 17.9 -> 29.1 mm, vias 3 -> 4
- net /APM_SPI1_CS: track 32.9 -> 25.2 mm
- net Net-(R9-Pad1): track 3.60 -> 6.59 mm
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Other:
- board text removed: "CS"
- board text removed: "MISO"
- board text removed: "MOSI"
