File: schematic/APM_v3_r1/APM.kicad_sch (KiCad schematic)
At the start: 36 parts, among them J1 ACM_CTRL, J10 Conn_02x17_Counter_Clockwise, J12 AUDIO_OUT, J13 Conn_02x36_Odd_Even, J14 periperhals, J15 Conn_02x36_Odd_Even, J2 CAN, J3 7SDD_CTRL, J4 LCD_display, J5 INTRPT, J6 Conn_02x10_Counter_Clockwise, J7 TDM_PMS_I2C, J8 Conn_02x15_Counter_Clockwise, J9 Conn_02x08_Counter_Clockwise, SW1 WARN_RST, SW2 FAIL_RST, U1 NUCLEO-H753ZI

Commit message: APM v3?
Connections:
- net APM_USB_D+: no longer J15.14 (Pin_14)
- net APM_USB_D-: no longer J15.12 (Pin_12)
- net APM_MIDI_RX: now reaches J13.57 (Pin_57)
- net APM_MIDI_RX: now also U1.CN11_57 (PD0)
- net APM_MIDI_TX: now reaches J13.59 (Pin_59)
- net APM_MIDI_TX: now also U1.CN11_55 (PD1)
- no-connect marks 322 -> 320
Other:
- sheet USB_MIDI_APM ports: added USB_MIDI_RX, USB_MIDI_TX; removed APM_MIDI_USB_D+, APM_MIDI_USB_D-
Changed lines of the file:
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@@
 	)
 	(no_connect
+		(at 328.93 55.88)
+	)
+	(no_connect
 		(at 309.88 171.45)
 	)
@@
 	)
 	(no_connect
-		(at 151.13 109.22)
-	)
-	(no_connect
 		(at 316.23 63.5)
 	)
@@
 	)
 	(no_connect
-		(at 223.52 116.84)
-	)
-	(no_connect
 		(at 223.52 132.08)
 	)
@@
 	)
 	(no_connect
-		(at 223.52 114.3)
-	)
-	(no_connect
 		(at 259.08 127)
 	)
@@
 	)
 	(no_connect
-		(at 151.13 106.68)
-	)
-	(no_connect
 		(at 236.22 66.04)
 	)
@@
 	)
 	(no_connect
+		(at 328.93 58.42)
+	)
+	(no_connect
 		(at 223.52 96.52)
 	)
@@
 	(wire
 		(pts
+			(xy 151.13 109.22) (xy 137.16 109.22)
+		)
+		(stroke
+			(width 0)
+			(type default)
+		)
+	)
+	(wire
+		(pts
 			(xy 250.19 81.28) (xy 236.22 81.28)
 		)
@@
 	(wire
 		(pts
+			(xy 118.11 64.77) (xy 132.08 64.77)
+		)
+		(stroke
+			(width 0)
+			(type default)
+		)
+	)
+	(wire
+		(pts
 			(xy 85.09 85.09) (xy 85.09 82.55)
 		)
@@
 	(wire
 		(pts
+			(xy 223.52 114.3) (xy 209.55 114.3)
+		)
+		(stroke
+			(width 0)
+			(type default)
+		)
+	)
+	(wire
+		(pts
 			(xy 77.47 172.72) (xy 96.52 172.72)
 		)
@@
 	(wire
 		(pts
-			(xy 176.53 172.72) (xy 166.37 172.72)
+			(xy 151.13 106.68) (xy 137.16 106.68)
 		)
 		(stroke
@@
 	(wire
 		(pts
-			(xy 342.9 55.88) (xy 328.93 55.88)
+			(xy 118.11 68.58) (xy 132.08 68.58)
+		)
+		(stroke
+			(width 0)
+			(type default)
+		)
+	)
+	(wire
+		(pts
+			(xy 176.53 172.72) (xy 166.37 172.72)
 		)
 		(stroke
@@
 	(wire
 		(pts
+			(xy 223.52 116.84) (xy 209.55 116.84)
+		)
+		(stroke
+			(width 0)
+			(type default)
+		)
+	)
+	(wire
+		(pts
 			(xy 248.92 45.72) (xy 236.22 45.72)
 		)
@@
 	(wire
 		(pts
-			(xy 236.22 63.5) (xy 238.76 63.5)
+			(xy 236.22 63.5) (xy 243.84 63.5)
 		)
 		(stroke
@@
 	(wire
 		(pts
-			(xy 342.9 58.42) (xy 328.93 58.42)
-		)
-		(stroke
-			(width 0)
-			(type default)
-		)
-	)
-	(wire
-		(pts
 			(xy 303.53 48.26) (xy 316.23 48.26)
 		)
@@
 	(wire
 		(pts
-			(xy 118.11 64.77) (xy 130.81 64.77)
-		)
-		(stroke
-			(width 0)
-			(type default)
-		)
-	)
-	(wire
-		(pts
 			(xy 344.17 83.82) (xy 328.93 83.82)
 		)
@@
 	(wire
 		(pts
-			(xy 118.11 68.58) (xy 130.81 68.58)
-		)
-		(stroke
-			(width 0)
-			(type default)
-		)
-	)
-	(wire
-		(pts
 			(xy 210.82 45.72) (xy 223.52 45.72)
 		)
@@
 		)
 	)
+	(label "APM_MIDI_TX"
+		(at 137.16 109.22 0)
+		(effects
+			(font
+				(size 1.27 1.27)
+			)
+			(justify left bottom)
+		)
+	)
+	(label "APM_MIDI_RX"
+		(at 137.16 106.68 0)
+		(effects
+			(font
+				(size 1.27 1.27)
+			)
+			(justify left bottom)
+		)
+	)
 	(label "APM_LED_FAIL"
 		(at 344.17 83.82 180)
@@
 		)
 	)
-	(label "APM_USB_D-"
-		(at 130.81 68.58 180)
-		(effects
-			(font
-				(size 1.27 1.27)
-			)
-			(justify right bottom)
-		)
-	)
 	(label "THRM_A"
 		(at 87.63 114.3 0)
@@
 		)
 	)
+	(label "APM_MIDI_TX"
+		(at 209.55 116.84 0)
+		(effects
+			(font
+				(size 1.27 1.27)
+			)
+			(justify left bottom)
+		)
+	)
 	(label "APM_CAN_TD"
 		(at 151.13 177.8 180)
@@
 		)
 	)
-	(label "APM_USB_D+"
-		(at 130.81 64.77 180)
-		(effects
-			(font
-				(size 1.27 1.27)
-			)
-			(justify right bottom)
-		)
-	)
 	(label "TDM_SCL"
 		(at 85.09 82.55 180)
@@
 		)
 	)
-	(label "APM_USB_D-"
-		(at 342.9 55.88 180)
-		(effects
-			(font
-				(size 1.27 1.27)
-			)
-			(justify right bottom)
-		)
-	)
 	(label "7SDD_CMD_TX"
 		(at 91.44 177.8 180)
@@
 		)
 	)
+	(label "APM_MIDI_RX"
+		(at 132.08 64.77 180)
+		(effects
+			(font
+				(size 1.27 1.27)
+			)
+			(justify right bottom)
+		)
+	)
 	(label "APM_WARN_RST"
 		(at 213.36 205.74 0)
@@
 		)
 	)
+	(label "APM_MIDI_TX"
+		(at 132.08 68.58 180)
+		(effects
+			(font
+				(size 1.27 1.27)
+			)
+			(justify right bottom)
+		)
+	)
 	(label "APM_LED_FAIL"
 		(at 346.71 104.14 0)
@@
 		)
 	)
+	(label "APM_MIDI_RX"
+		(at 209.55 114.3 0)
+		(effects
+			(font
+				(size 1.27 1.27)
+			)
+			(justify left bottom)
+		)
+	)
 	(label "POT_2"
 		(at 243.84 88.9 180)
@@
 		)
 	)
-	(label "APM_USB_D+"
-		(at 342.9 58.42 180)
-		(effects
-			(font
-				(size 1.27 1.27)
-			)
-			(justify right bottom)
-		)
-	)
 	(label "POT_4"
 		(at 308.61 88.9 0)
@@
 	(symbol
 		(lib_id "power:+5V")
-		(at 238.76 63.5 0)
+		(at 243.84 63.5 0)
 		(unit 1)
 		(exclude_from_sim no)
@@
 		(fields_autoplaced yes)
 		(property "Reference" "#PWR016"
-			(at 238.76 67.31 0)
+			(at 243.84 67.31 0)
 			(effects
 				(font
@@
 		)
 		(property "Value" "5V_APM_MCU"
-			(at 238.76 58.42 0)
+			(at 243.84 58.42 0)
 			(effects
 				(font
@@
 		)
 		(property "Footprint" ""
-			(at 238.76 63.5 0)
+			(at 243.84 63.5 0)
 			(effects
 				(font
@@
 		)
 		(property "Datasheet" ""
-			(at 238.76 63.5 0)
+			(at 243.84 63.5 0)
 			(effects
 				(font
@@
 		)
 		(property "Description" "Power symbol creates a global label with name \"+5V\""
-			(at 238.76 63.5 0)
+			(at 243.84 63.5 0)
 			(effects
 				(font
@@
 		)
 		(property "Value" "GND"
-			(at 242.57 55.88 0)
+			(at 245.11 52.0699 0)
 			(effects
 				(font
 					(size 1.27 1.27)
 				)
+				(justify left)
 			)
 		)
@@
 		)
 		(property "Value" "3V3_APM_MCU"
-			(at 248.92 59.6899 0)
+			(at 246.38 55.88 0)
 			(effects
 				(font
 					(size 1.27 1.27)
 				)
-				(justify left)
 			)
 		)
@@
 			)
 		)
-		(pin "APM_MIDI_USB_D+" bidirectional
-			(at 118.11 64.77 0)
+		(pin "USB_MIDI_RX" input
+			(at 118.11 68.58 0)
 			(effects
 				(font
@@
 			)
 		)
-		(pin "APM_MIDI_USB_D-" bidirectional
-			(at 118.11 68.58 0)
+		(pin "USB_MIDI_TX" output
+			(at 118.11 64.77 0)
 			(effects
 				(font

Commit message: updating top v10. need to get 3v3 APM converged in schematic. routing is tricky right now. the components should be evenly laid out and have the NUCLEO pins be adjusted based on location
Parts:
- removed J12: AUDIO_OUT, Connector_PinHeader_2.54mm:PinHeader_1x03_P2.54mm_Vertical, symbol Connector_Generic:Conn_01x04
- removed J15: Conn_02x36_Odd_Even, Connector_PinHeader_1.00mm:PinHeader_2x36_P1.00mm_Vertical, symbol Connector_Generic:Conn_02x36_Odd_Even
- removed J7: TDM_PMS_I2C, Connector_PinHeader_1.00mm:PinHeader_1x02_P1.00mm_Vertical, symbol Connector_Generic:Conn_01x02
- removed R1, R2: 300, Resistor_SMD:R_0805_2012Metric_Pad1.20x1.40mm_HandSolder, symbol Device:R
- removed R3: 10k, Resistor_SMD:R_0805_2012Metric_Pad1.20x1.40mm_HandSolder, symbol Device:R
- removed R4: 20k, Resistor_SMD:R_0805_2012Metric_Pad1.20x1.40mm_HandSolder, symbol Device:R
- removed SW1: WARN_RST, Button_Switch_SMD:SW_SPST_FSMSM, symbol Switch:SW_Push
- removed SW2: FAIL_RST, Button_Switch_SMD:SW_SPST_FSMSM, symbol Switch:SW_Push
- removed TP1: DAC_R_TP, TestPoint:TestPoint_THTPad_D2.5mm_Drill1.2mm, symbol Connector:TestPoint
- removed TP2: DAC_L_TP, TestPoint:TestPoint_THTPad_D2.5mm_Drill1.2mm, symbol Connector:TestPoint
- removed TP4: THRM_B, TestPoint:TestPoint_Pad_1.5x1.5mm, symbol Connector:TestPoint
- removed TP6: THRM_D, TestPoint:TestPoint_Pad_1.5x1.5mm, symbol Connector:TestPoint
- added J11: DAC_L_PRB, Connector_Coaxial:U.FL_Hirose_U.FL-R-SMT-1_Vertical, symbol Connector:Conn_Coaxial_Small
- added J12: Conn_01x02, Connector_PinHeader_2.54mm:PinHeader_1x02_P2.54mm_Vertical, symbol Connector_Generic:Conn_01x02
- added J15: FPGA FFC, Connector_FFC-FPC:Hirose_FH12-40S-0.5SH_1x40-1MP_P0.50mm_Horizontal, symbol Connector_Generic:Conn_01x40
- added J18: Conn_02x36_Odd_Even, Connector_PinSocket_2.54mm:PinSocket_2x36_P2.54mm_Vertical, symbol Connector_Generic:Conn_02x36_Odd_Even
- added J7: DAC_R_PRB, Connector_Coaxial:U.FL_Hirose_U.FL-R-SMT-1_Vertical, symbol Connector:Conn_Coaxial_Small
- J13: footprint Connector_PinHeader_1.00mm:PinHeader_2x36_P1.00mm_Vertical -> Connector_PinSocket_2.54mm:PinSocket_2x36_P2.54mm_Vertical
- J14: value periperhals -> ADC FFC
- R38: value 300 -> 1.2k; footprint Resistor_SMD:R_0805_2012Metric_Pad1.20x1.40mm_HandSolder -> Resistor_SMD:R_0201_0603Metric
- R39, R40, R41: footprint Resistor_SMD:R_0805_2012Metric_Pad1.20x1.40mm_HandSolder -> Resistor_SMD:R_0201_0603Metric
Connections:
- net APM_DAC_L is gone; now on net DAC_1-2_L: U1.CN12_11 (PA5)
- net 3V3_APM: now also J14.9 (Pin_9); no longer J14.6 (Pin_6)
- net 3V3_APM_MCU: now also J18.16 (Pin_16); no longer J13.16 (Pin_16)
- net 5V_APM: no longer J14.9 (Pin_9)
- net 5V_APM_MCU: now also J18.18 (Pin_18); no longer J13.18 (Pin_18)
- net 7SDD_CMD_RX: now also J13.65 (Pin_65); no longer J13.63 (Pin_63)
- net 7SDD_CMD_TX: now also J13.66 (Pin_66)
- net APM_CAN_RD: now also J13.3 (Pin_3)
- net APM_CAN_TD: now also J13.5 (Pin_5)
- net APM_CMD_RX: now also J18.2 (Pin_2); no longer J13.2 (Pin_2)
- net APM_CMD_TX: now also J18.1 (Pin_1); no longer J13.1 (Pin_1)
- net APM_DBG_RX: now also J18.4 (Pin_4); no longer J13.4 (Pin_4)
- net APM_DBG_TX: now also J18.3 (Pin_3); no longer J13.3 (Pin_3)
- net APM_FAIL_RST: now also J13.2 (Pin_2)
- net APM_I2C1_SCL: no longer J13.51 (Pin_51), J4.3 (Pin_3)
- net APM_I2C1_SDA: no longer J13.53 (Pin_53), J4.2 (Pin_2)
- net APM_IRQ0: now also J13.71 (Pin_71); no longer J13.62 (Pin_62)
- net APM_ISR0: now also J13.69 (Pin_69); no longer J13.47 (Pin_47)
- net APM_LED_FAIL: now also J13.68 (Pin_68)
- net APM_LED_OK: now also J13.70 (Pin_70)
- net APM_LED_WARN: now also J13.72 (Pin_72)
- net APM_MIDI_RX: now also J18.57 (Pin_57); no longer J13.57 (Pin_57)
- net APM_MIDI_TX: now also J18.59 (Pin_59); no longer J13.59 (Pin_59)
- net APM_USB_D+: now also J13.14 (Pin_14)
- net APM_USB_D-: now also J13.12 (Pin_12)
- net APM_WARN_RST: now also J13.1 (Pin_1)
- net GND: now also J13.56 (Pin_56), J13.9 (Pin_9), J14.2 (Pin_2), J14.4 (Pin_4), J14.6 (Pin_6), J14.8 (Pin_8), J11.2 (Ext), J15.13 (Pin_13), J15.14 (Pin_14), J15.21 (Pin_21), J15.22 (Pin_22), J15.23 (Pin_23), J15.29 (Pin_29), J15.3 (Pin_3), J15.36 (Pin_36), J15.5 (Pin_5), J15.6 (Pin_6), J15.7 (Pin_7), J18.8 (Pin_8), J7.2 (Ext); no longer J13.8 (Pin_8)
- net ADC_1-10_POT_3: now reaches J14.5 (Pin_5)
- net ADC_1-10_POT_3: now also J18.36 (Pin_36)
- net ADC_3-1_POT_4: now reaches J14.7 (Pin_7)
- net ADC_3-1_POT_4: now also J18.35 (Pin_35)
- net DAC_1-2_L: now reaches J13.11 (Pin_11)
- net DAC_1-2_L: now also J11.1 (In), J12.1 (Pin_1)
- net APM_DAC_R: no longer names the net of J13.32 (Pin_32)
- net APM_DAC_R: no longer U1.CN11_32 (PA4)
- net POT_1: no longer names the net of U1.CN12_24 (PB1)
- net POT_1: no longer J14.1 (Pin_1)
- removed net POT_2: J13.38 (Pin_38), J14.2 (Pin_2), U1.CN11_38 (PC0)
- removed net POT_3: J13.37 (Pin_37), J14.3 (Pin_3), U1.CN11_37 (PC3)
- net POT_4: no longer names the net of U1.CN12_37 (PA3)
- net POT_4: no longer J14.4 (Pin_4)
- new net ADC_1-16_POT_1: J14.1 (Pin_1), J18.30 (Pin_30)
- new net ADC_1-5_POT_2: J14.3 (Pin_3), J18.34 (Pin_34)
- new net APM_EEPROM_EN: J18.68 (Pin_68)
- new net APM_I2C2_SCL: J18.51 (Pin_51), J4.3 (Pin_3)
- new net APM_I2C2_SDA: J18.53 (Pin_53), J4.2 (Pin_2)
- new net APM_MRAM_EN: J18.66 (Pin_66)
- new net APM_SPI1_MISO: J18.65 (Pin_65)
- new net APM_SPI1_MOSI: J18.47 (Pin_47)
- new net APM_SPI1_SCK: J18.72 (Pin_72)
- new net APM_SPIFLASH_EN: J18.64 (Pin_64)
- new net DAC_1-1_R: J12.2 (Pin_2), J18.32 (Pin_32), J7.1 (In), U1.CN11_32 (PA4)
- new net FPGA_3V3_OUT1: J15.31 (Pin_31), J15.4 (Pin_4)
- new net SPIFLASH_CS: J18.69 (Pin_69)
- new net SPIMRAM_CS: J18.71 (Pin_71)
- no-connect marks 320 -> 309
Other:
- added sheet STORAGE_APM (STORAGE_APM.kicad_sch)
- sheet PMS_APM ports: added 3V3_OUT, APM_I2C1_SCL, APM_I2C1_SDA; removed TDM_I2C1_SCL, TDM_I2C1_SDA
- sheet THERMISTORS_APM ports: added none; removed THERMISTOR_B, THERMISTOR_D
- note added: "NOT ROUTED, FOR REFERENCE ONLY"
- moved on the sheet: D15, D16, D17, D18, J1, J10, J14, J2, J3, J4, J5, J6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

Commit message: i got orientation wrong big time
Connections:
- net 5V_APM_MCU: now also J13.17 (Pin_17)
- net 7SDD_CMD_RX: no longer J13.65 (Pin_65)
- net 7SDD_CMD_TX: no longer J13.66 (Pin_66)
- net ADC_1-10_POT_3: now also J13.35 (Pin_35); no longer J18.36 (Pin_36)
- net ADC_1-16_POT_1: now also J13.29 (Pin_29); no longer J18.30 (Pin_30)
- net ADC_1-5_POT_2: now also J13.33 (Pin_33); no longer J18.34 (Pin_34)
- net ADC_3-1_POT_4: now also J13.36 (Pin_36); no longer J18.35 (Pin_35)
- net APM_CAN_RD: no longer J13.3 (Pin_3)
- net APM_CAN_TD: no longer J13.5 (Pin_5)
- net APM_EEPROM_EN: no longer J18.68 (Pin_68)
- net APM_FAIL_RST: no longer J13.2 (Pin_2)
- net APM_IRQ0: no longer J13.71 (Pin_71)
- net APM_ISR0: no longer J13.69 (Pin_69)
- net APM_LED_FAIL: now also J18.68 (Pin_68); no longer J13.68 (Pin_68)
- net APM_LED_OK: now also J18.70 (Pin_70); no longer J13.70 (Pin_70)
- net APM_LED_WARN: now also J18.72 (Pin_72); no longer J13.72 (Pin_72)
- net APM_MIDI_RX: no longer J18.57 (Pin_57)
- net APM_MIDI_TX: no longer J18.59 (Pin_59)
- net APM_MRAM_EN: no longer J18.66 (Pin_66)
- net APM_SPI1_MISO: no longer J18.65 (Pin_65)
- net APM_SPI1_MOSI: no longer J18.47 (Pin_47)
- net APM_SPI1_SCK: no longer J18.72 (Pin_72)
- net APM_SPIFLASH_EN: no longer J18.64 (Pin_64)
- net APM_USB_D+: no longer J13.14 (Pin_14)
- net APM_USB_D-: no longer J13.12 (Pin_12)
- net APM_WARN_RST: no longer J13.1 (Pin_1)
- net DAC_1-1_R: now also J13.31 (Pin_31); no longer J18.32 (Pin_32)
- net DAC_1-2_L: no longer J13.11 (Pin_11)
- net GND: now also J13.19 (Pin_19), J13.21 (Pin_21), J13.61 (Pin_61), J13.7 (Pin_7); no longer J13.56 (Pin_56), J13.9 (Pin_9)
- net SPIFLASH_CS: no longer J18.69 (Pin_69)
- net SPIMRAM_CS: no longer J18.71 (Pin_71)
- new net UART3_RX: J13.1 (Pin_1)
- new net UART3_TX: J13.2 (Pin_2)
- no-connect marks 309 -> 317
Other:
- note added: "CN11"
- note added: "CN12"
- note added: "INSIDE"
- note added: "NOTE: these pins mirror the NUCLEO-144 GPIOs if it were to be facing north/upwards. Our board attaches to the "bottom" of the NUCLEO."
- note removed: "TODO: verify these pinouts on MCU"
- moved on the sheet: J10, J13, J18, J6, J8, J9, U1B

Commit message: more progress
Parts:
- added D19: FPGA_PWR, LED_SMD:LED_0603_1608Metric, symbol Device:LED
- added R42: 300, Resistor_SMD:R_0201_0603Metric, symbol Device:R
Connections:
- net UART3_RX is gone; now on net APM_MIDI_RX: J13.1 (Pin_1)
- net UART3_TX is gone; now on net APM_MIDI_TX: J13.2 (Pin_2)
- net 3V3_APM_MCU: no longer J18.16 (Pin_16)
- net 5V_APM_MCU: no longer J18.18 (Pin_18)
- net 7SDD_CMD_RX: now also J13.46 (Pin_46)
- net 7SDD_CMD_TX: now also J13.44 (Pin_44); no longer U1.CN12_61 (PG14)
- net ADC_1-10_POT_3: no longer J14.5 (Pin_5)
- net ADC_1-16_POT_1: no longer J14.1 (Pin_1)
- net ADC_1-5_POT_2: no longer J14.3 (Pin_3)
- net ADC_3-1_POT_4: no longer J14.7 (Pin_7)
- net APM_CAN_RD: now also J18.13 (Pin_13), U1.CN12_53 (PE15); no longer U1.CN12_3 (PB8)
- net APM_CAN_TD: now also J18.11 (Pin_11); no longer U1.CN12_5 (PB9)
- net APM_CMD_RX: now also J18.4 (Pin_4); no longer J18.2 (Pin_2)
- net APM_CMD_TX: now also J18.6 (Pin_6); no longer J18.1 (Pin_1)
- net APM_DBG_RX: now also J18.17 (Pin_17); no longer J18.4 (Pin_4)
- net APM_DBG_TX: now also J18.9 (Pin_9); no longer J18.3 (Pin_3)
- net APM_EEPROM_EN: now also J13.68 (Pin_68)
- net APM_FAIL_RST: now also U1.CN12_68 (PG5); no longer U1.CN12_2 (PC8)
- net APM_I2C2_SCL: now also J13.54 (Pin_54), J15.9 (Pin_9); no longer J18.51 (Pin_51)
- net APM_I2C2_SDA: now also J13.56 (Pin_56), J15.8 (Pin_8); no longer J18.53 (Pin_53)
- net APM_IRQ0: now also J13.72 (Pin_72)
- net APM_ISR0: now also J13.71 (Pin_71)
- net APM_LED_FAIL: now also J13.65 (Pin_65); no longer J18.68 (Pin_68), U1.CN12_34 (PC4)
- net APM_LED_OK: now also J13.67 (Pin_67); no longer J18.70 (Pin_70), U1.CN12_4 (PC6)
- net APM_LED_WARN: now also J13.69 (Pin_69); no longer J18.72 (Pin_72), U1.CN12_6 (PC5)
- net APM_MRAM_EN: now also J13.66 (Pin_66)
- net APM_SPI1_MISO: now also J15.15 (Pin_15)
- net APM_SPI1_MOSI: now also J15.16 (Pin_16)
- net APM_SPIFLASH_EN: now also J13.64 (Pin_64)
- net APM_USB_D+: now also U1.CN12_64 (PE0); no longer U1.CN12_14 (PA11)
- net APM_USB_D-: now also U1.CN12_44 (PE7); no longer U1.CN12_12 (PA12)
- net APM_WARN_RST: now also U1.CN12_70 (PG6); no longer U1.CN12_1 (PC9)
- net DAC_1-2_L: now also J18.12 (Pin_12), U1.CN12_45 (PD11); no longer U1.CN12_11 (PA5)
- net FPGA_3V3_OUT1: now also R42.2
- net GND: now also J13.20 (Pin_20), J13.52 (Pin_52), J15.11 (Pin_11), J15.27 (Pin_27), J15.32 (Pin_32), J15.38 (Pin_38), J18.10 (Pin_10), J18.66 (Pin_66), D19.1 (K); no longer J18.8 (Pin_8)
- net SPIFLASH_CS: now also J13.51 (Pin_51)
- net SPIMRAM_CS: now also J13.53 (Pin_53)
- net ADC_3-6_POT_4: now reaches J18.44 (Pin_44)
- net ADC_3-6_POT_4: now also J14.7 (Pin_7)
- net ADC_1-2_POT_1: now reaches J18.59 (Pin_59)
- net ADC_1-2_POT_1: now also J14.1 (Pin_1)
- net ADC_3-5_POT_3: now reaches J18.60 (Pin_60)
- net ADC_3-5_POT_3: now also J14.5 (Pin_5)
- net ADC_2-2_POT_2: now reaches J18.61 (Pin_61)
- net ADC_2-2_POT_2: now also J14.3 (Pin_3)
- net APM_SPI1_CLK: now reaches J15.12 (Pin_12)
- net APM_SPI1_CS: now reaches J15.17 (Pin_17)
- net APM_FPGA_UART_TX: now reaches J15.25 (Pin_25)
- net APM_FPGA_UART_RX: now reaches J15.26 (Pin_26)
- net QSPI_NCS: now reaches J15.28 (Pin_28)
- net GCLKT_1: now reaches J15.30 (Pin_30)
- net QSPI_IO_3: now reaches J15.33 (Pin_33)
- net QSPI_IO_2: now reaches J15.34 (Pin_34)
- net QSPI_IO_1: now reaches J15.39 (Pin_39)
- net QSPI_IO_0: now reaches J15.40 (Pin_40)
- net NC: now reaches J13.25 (Pin_25)
- net NC: now also J13.26 (Pin_26), J13.28 (Pin_28), J13.30 (Pin_30), J13.70 (Pin_70)
- net UART5_RX: now reaches J13.3 (Pin_3)
- net UART5_TX: now reaches J13.4 (Pin_4)
- net APM_SPI4_SCK: now reaches J13.45 (Pin_45)
- net APM_SPI4_MISO: now reaches J13.49 (Pin_49)
- net SPIFPGA_CS: now reaches J13.55 (Pin_55)
- net APM_SPI4_MOSI: now reaches J13.63 (Pin_63)
- new net: D19.2 (A), R42.1
- no-connect marks 317 -> 294

Commit message: more routing
Connections:
- net APM_CAN_RD: now also U1.CN12_3 (PB8); no longer U1.CN12_53 (PE15)
- net APM_CAN_TD: now also U1.CN12_5 (PB9)
- net APM_FAIL_RST: now also U1.CN12_2 (PC8); no longer U1.CN12_68 (PG5)
- net APM_USB_D+: now also U1.CN12_14 (PA11); no longer U1.CN12_64 (PE0)
- net APM_USB_D-: now also U1.CN12_12 (PA12); no longer U1.CN12_44 (PE7)
- net APM_WARN_RST: now also U1.CN12_1 (PC9); no longer U1.CN12_70 (PG6)
- net DAC_1-2_L: now also U1.CN12_11 (PA5); no longer U1.CN12_45 (PD11)
- no-connect marks 294 -> 290
Changed lines of the file:
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@@
 	)
 	(no_connect
-		(at 401.32 128.27)
-	)
-	(no_connect
 		(at 270.51 97.79)
 	)
@@
 	)
 	(no_connect
-		(at 401.32 125.73)
-	)
-	(no_connect
 		(at 222.25 74.93)
 	)
@@
 	)
 	(no_connect
-		(at 401.32 118.11)
-	)
-	(no_connect
 		(at 365.76 107.95)
 	)
@@
 		(at 257.81 105.41)
 	)
-	(no_connect
-		(at 401.32 115.57)
-	)
 	(wire
 		(pts
@@
 	(wire
 		(pts
-			(xy 401.32 120.65) (xy 415.29 120.65)
-		)
-		(stroke
-			(width 0)
-			(type default)
-		)
-	)
-	(wire
-		(pts
 			(xy 314.96 36.83) (xy 308.61 36.83)
 		)
@@
 		)
 	)
-	(label "7SDD_CMD_TX"
-		(at 415.29 120.65 180)
-		(effects
-			(font
-				(size 1.27 1.27)
-			)
-			(justify right bottom)
-		)
-	)
 	(label "APM_DBG_TX"
 		(at 113.03 29.21 180)
@@
 		(lib_id "NUCLEO-H753ZI:NUCLEO-H753ZI")
 		(at 383.54 77.47 0)
-		(mirror y)
 		(unit 2)
 		(body_style 1)
@@
 		(in_pos_files yes)
 		(dnp no)
-		(fields_autoplaced yes)
 		(property "Reference" "U1"
 			(at 383.54 16.51 0)

Commit message: ground planes on f and b cu
Parts:
- added J19: FPGA_QSPI, Connector_PinHeader_2.54mm:PinHeader_1x06_P2.54mm_Vertical, symbol Connector_Generic:Conn_01x06
- added J20: FPGA_UART, Connector_PinHeader_2.54mm:PinHeader_1x02_P2.54mm_Vertical, symbol Connector_Generic:Conn_01x02
- added J21: APM_FPGA_UART, Connector_PinHeader_2.54mm:PinHeader_1x02_P2.54mm_Vertical, symbol Connector_Generic:Conn_01x02
- added J22: FPGA_SPI, Connector_PinHeader_2.54mm:PinHeader_1x04_P2.54mm_Vertical, symbol Connector_Generic:Conn_01x04
Connections:
- net ADC_1-10_POT_3 is gone; now on net SPIMRAM_CS: J13.35 (Pin_35)
- net ADC_1-5_POT_2 is gone; now on net SPIFLASH_CS: J13.33 (Pin_33)
- net APM_EEPROM_EN: now also J13.42 (Pin_42); no longer J13.68 (Pin_68)
- net APM_FPGA_UART_RX: now also J21.2 (Pin_2)
- net APM_FPGA_UART_TX: now also J21.1 (Pin_1)
- net APM_MRAM_EN: now also J13.37 (Pin_37); no longer J13.66 (Pin_66)
- net APM_SPI1_CLK: now also J22.1 (Pin_1)
- net APM_SPI1_CS: now also J22.4 (Pin_4)
- net APM_SPI1_MISO: now also J22.2 (Pin_2)
- net APM_SPI1_MOSI: now also J22.3 (Pin_3)
- net APM_SPIFLASH_EN: now also J13.39 (Pin_39); no longer J13.64 (Pin_64)
- net GCLKT_1: now also J19.2 (Pin_2)
- net QSPI_IO_0: now also J19.6 (Pin_6)
- net QSPI_IO_1: now also J19.5 (Pin_5)
- net QSPI_IO_2: now also J19.4 (Pin_4)
- net QSPI_IO_3: now also J19.3 (Pin_3)
- net QSPI_NCS: now also J19.1 (Pin_1)
- net SPIFLASH_CS: no longer J13.51 (Pin_51)
- net SPIFPGA_CS: now also J13.59 (Pin_59); no longer J13.55 (Pin_55)
- net SPIMRAM_CS: no longer J13.53 (Pin_53)
- net FPGA_UART_TX: now reaches J15.35 (Pin_35)
- net FPGA_UART_TX: now also J20.1 (Pin_1)
- net FPGA_UART_RX: now reaches J15.37 (Pin_37)
- net FPGA_UART_RX: now also J20.2 (Pin_2)
- net ADC_1-16_POT_1: no longer names the net of J13.29 (Pin_29)
- net ADC_3-1_POT_4: no longer names the net of J13.36 (Pin_36)
- no-connect marks 290 -> 297
Other:
- sheet STORAGE_APM ports: added EEPROM_EN, EEPROM_SCL, EEPROM_SDA, SPIFLASH_EN, SPIFLASH_MISO, SPIFLASH_MOSI, SPIFLASH_SCK, SPIMRAM_EN, SPIMRAM_MISO, SPIMRAM_MOSI, SPIMRAM_SCK; removed APM_EEPROM_EN, APM_I2C2_SCL, APM_I2C2_SDA, APM_MRAM_EN, APM_SPI1_MISO, APM_SPI1_MOSI, APM_SPI1_SCK, APM_SPIFLASH_EN

Commit message: getting APM V3 R1 made. starting R2
Parts:
- removed J22: FPGA_SPI, Connector_PinHeader_2.54mm:PinHeader_1x04_P2.54mm_Vertical, symbol Connector_Generic:Conn_01x04
- added CLK1, CS1, MISO1, MOSI1: (no value), TestPoint:TestPoint_Pad_D1.0mm, symbol Connector:TestPoint
- added J23: QSPIFLASH, Connector_PinHeader_2.54mm:PinHeader_1x06_P2.54mm_Vertical, symbol Connector_Generic:Conn_01x06
Connections:
- net APM_SPI1_CLK: now also CLK1.1
- net APM_SPI1_CS: now also CS1.1
- net APM_SPI1_MISO: now also MISO1.1
- net APM_SPI1_MOSI: now also MOSI1.1
- new net STORAGE_APM/QSPIFLASH_CLK: J23.5 (Pin_5)
- new net STORAGE_APM/QSPIFLASH_CS: J23.1 (Pin_1)
- new net STORAGE_APM/QSPIFLASH_IO0: J23.6 (Pin_6)
- new net STORAGE_APM/QSPIFLASH_IO1: J23.2 (Pin_2)
- new net STORAGE_APM/QSPIFLASH_IO2: J23.3 (Pin_3)
- new net STORAGE_APM/QSPIFLASH_IO3: J23.4 (Pin_4)
Other:
- sheet STORAGE_APM ports: added QSPIFLASH_CLK, QSPIFLASH_CS, QSPIFLASH_IO0, QSPIFLASH_IO1, QSPIFLASH_IO2, QSPIFLASH_IO3; removed none
