File: schematic/APM_v3_r2/APM.kicad_sch (KiCad schematic)
At the start: 32 parts, among them J1 ACM_CTRL, J10 Conn_02x17_Counter_Clockwise, J11 DAC_L_PRB, J12 Conn_01x02, J13 Conn_01x06, J14 PERIPH_FFC, J15 FPGA FFC, J2 CAN, J20 FPGA_UART, J21 APM_FPGA_UART, J3 7SDD_CTRL, J4 LCD_display, J5 INTRPT, J6 Conn_02x10_Counter_Clockwise, J7 DAC_R_PRB, J8 Conn_02x15_Counter_Clockwise, J9 Conn_02x08_Counter_Clockwise

Commit message: routed
Parts:
- removed J11: DAC_L_PRB, Connector_Coaxial:U.FL_Hirose_U.FL-R-SMT-1_Vertical, symbol Connector:Conn_Coaxial_Small
- removed J12: Conn_01x02, Connector_PinHeader_2.54mm:PinHeader_1x02_P2.54mm_Vertical, symbol Connector_Generic:Conn_01x02
- removed J7: DAC_R_PRB, Connector_Coaxial:U.FL_Hirose_U.FL-R-SMT-1_Vertical, symbol Connector:Conn_Coaxial_Small
Connections:
- net APM_SPI1_CS: now also J15.12 (Pin_12); no longer J15.9 (Pin_9)
- net APM_SPI1_MISO: now also J15.9 (Pin_9); no longer J15.12 (Pin_12)
- net APM_SPI1_MOSI: now also J15.8 (Pin_8); no longer J15.15 (Pin_15)
- net APM_SPI1_SCK: now also J15.15 (Pin_15); no longer J15.8 (Pin_8)
Other:
- added sheet AUDIO_APM (AUDIO_APM.kicad_sch)

Commit message: routing changes
Parts:
- removed J3: 7SDD_CTRL, Connector_PinHeader_2.54mm:PinHeader_1x03_P2.54mm_Vertical, symbol Connector_Generic:Conn_01x03
- removed J5: INTRPT, Connector_PinHeader_2.54mm:PinHeader_1x02_P2.54mm_Vertical, symbol Connector_Generic:Conn_01x02
- added C17: 100nF, Capacitor_SMD:C_0805_2012Metric, symbol Device:C_Small
Connections:
- net 5V_APM: now also C17.2
- net GND: now also C17.1

Commit message: v4 with new FFC conn
Parts:
- removed J21: APM_FPGA_UART, Connector_PinHeader_2.54mm:PinHeader_1x02_P2.54mm_Vertical, symbol Connector_Generic:Conn_01x02
- added J18: CTRL_FFC, Connector_FFC-FPC:Hirose_FH12-10S-0.5SH_1x10-1MP_P0.50mm_Horizontal, symbol Connector_Generic:Conn_01x10
- J14: value PERIPH_FFC -> POT_FFC
Connections:
- net 3V3_APM: now also J18.1 (Pin_1), J18.10 (Pin_10)
- net APM_FPGA_UART_RX: now also J15.25 (Pin_25), U10.44 (PE7); no longer J15.26 (Pin_26)
- net APM_FPGA_UART_TX: now also J15.26 (Pin_26), U10.40 (PE8); no longer J15.25 (Pin_25)
- net GND: now also J18.2 (Pin_2), J18.6 (Pin_6), J18.9 (Pin_9)
- net SR_GPIO1: now reaches U10.13 (PA6)
- net SR_GPIO1: now also J18.4 (Pin_4)
- net SR_GPIO2: now reaches U10.15 (PA7)
- net SR_GPIO2: now also J18.7 (Pin_7)
- net APM_SPI4_SCK: now reaches U10.49 (PE12)
- net APM_SPI4_SCK: now also J18.3 (Pin_3)
- net APM_SPI4_MOSI: now reaches U10.51 (PE14)
- net APM_SPI4_MOSI: now also J18.8 (Pin_8)
- net APM_SPI4_MISO: now reaches U10.55 (PE13)
- net APM_SPI4_MISO: now also J18.5 (Pin_5)
- no-connect marks 157 -> 140
Other:
- moved on the sheet: J13, J14, J20
