File: schematic/APM_v3_r2/AUDIO_APM.kicad_sch (KiCad schematic)
At the start: 15 parts, among them U13 INA219AxD, U3 LT1963AxST-3.3, U7 INA219AxD

Commit message: routed
Parts:
- removed C5, C7: 0.1uf, Capacitor_SMD:C_0805_2012Metric, symbol Device:C_Small
- removed C9: 100nF, Capacitor_SMD:C_0805_2012Metric, symbol Device:C_Small
- removed D5, D7: LED_PWR, LED_SMD:LED_0603_1608Metric, symbol Device:LED
- removed R15, R30: 300, Resistor_SMD:R_0201_0603Metric, symbol Device:R
- removed R16, R3: 0.1, Resistor_SMD:R_Shunt_Ohmite_LVK12, symbol Device:R_Shunt
- removed R26, R28, R4: 10k, Resistor_SMD:R_0201_0603Metric, symbol Device:R
- removed U13, U7: INA219AxD, Package_SO:SOIC-8_3.9x4.9mm_P1.27mm, symbol Sensor_Energy:INA219AxD
- removed U3: LT1963AxST-3.3, Package_TO_SOT_SMD:SOT-223-3_TabPin2, symbol Regulator_Linear:LT1963AxST-3.3
- added C10, C12: 2.2nF, Capacitor_SMD:C_0805_2012Metric, symbol Device:C_Small
- added C11, C13: 4.7nF, Capacitor_SMD:C_0805_2012Metric, symbol Device:C_Small
- added C14, C15, C2: 10uF, Capacitor_SMD:CP_Elec_4x3, symbol Device:C_Small
- added C3: 100nF, Capacitor_SMD:C_0805_2012Metric, symbol Device:C_Small
- added J11: DAC_L_PRB, Connector_Coaxial:U.FL_Hirose_U.FL-R-SMT-1_Vertical, symbol Connector:Conn_Coaxial_Small
- added J12: Conn_01x02, Connector_PinHeader_2.54mm:PinHeader_1x02_P2.54mm_Vertical, symbol Connector_Generic:Conn_01x02
- added J19: AudioPlug3, Connector_Audio:Jack_3.5mm_Ledino_KB3SPRS_Horizontal, symbol Connector_Audio:AudioPlug3
- added J23: VOL_L_CTRL, Connector_PinHeader_2.54mm:PinHeader_1x03_P2.54mm_Vertical, symbol Connector_Generic:Conn_01x03
- added J24: VOL_R_CTRL, Connector_PinHeader_2.54mm:PinHeader_1x03_P2.54mm_Vertical, symbol Connector_Generic:Conn_01x03
- added J7: DAC_R_PRB, Connector_Coaxial:U.FL_Hirose_U.FL-R-SMT-1_Vertical, symbol Connector:Conn_Coaxial_Small
- added R43, R44, R45, R46: 2.4k, Resistor_SMD:R_0201_0603Metric, symbol Device:R
- added R47, R48: 47, Resistor_SMD:R_0201_0603Metric, symbol Device:R
- added U2: OPA1678, Package_DIP:DIP-8_W7.62mm_SMDSocket_SmallPads, symbol Amplifier_Operational:OPA1678
Connections:
- net GND: now also C10.1, C12.1, C2.1, C3.1, J11.2 (Ext), J19.S, J23.3 (Pin_3), J24.3 (Pin_3), J7.2 (Ext), U2.4 (V-)
- new net: C10.2, R45.2, U2.3 (+)
- new net: C11.2, R43.2, R45.1
- new net: C13.2, R44.2, R46.1
- new net: J19.R, R48.1
- new net: J19.T, R47.1
- new net: C12.2, R46.2, U2.5 (+)
- new net 5V_APM: C2.2, C3.2, U2.8 (V+)
- new net DAC_L_IN: J11.1 (In), J12.1 (Pin_1), R43.1
- new net DAC_L_OUT: C11.1, C14.2, U2.1, U2.2 (-)
- new net DAC_R_IN: J12.2 (Pin_2), J7.1 (In), R44.1
- new net DAC_R_OUT: C13.1, C15.2, U2.6 (-), U2.7
- new net OUT_L: J23.2 (Pin_2), R47.2
- new net OUT_R: J24.2 (Pin_2), R48.2
- new net VOL_L_IN: C14.1, J23.1 (Pin_1)
- new net VOL_R_IN: C15.1, J24.1 (Pin_1)
Other:
- note removed: "3v3 INA219 APM"
- note removed: "5v INA219 APM"
- note removed: "I2C addr: 0x40"
- note removed: "I2C addr: 0x41"
- note removed: "PMS has an INA219 current sensor for each board/node in the PCB. Each takes in the 5V from it's parent board and supplies 5V to said board's circuit (its peripherals) thus enabling monitoring"
- note removed: "Power Monitor and Supply"

Commit message: routing changes
Parts:
- added TP1: DAC_R, TestPoint:TestPoint_Pad_D1.0mm, symbol Connector:TestPoint
- added TP2: DAC_L, TestPoint:TestPoint_Pad_D1.0mm, symbol Connector:TestPoint
- added U11: PCM5102A, Package_SO:TSSOP-20_4.4x6.5mm_P0.65mm, symbol Audio:PCM5102A
Connections:
- net DAC_L_OUT: now also TP2.1
- net DAC_R_OUT: now also TP1.1
Other:
- moved on the sheet: C10, C11, C12, C13, C14, C15, C2, C3, J11, J12, J19, J23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

Commit message: v4 with new FFC conn
Parts:
- removed U11: PCM5102A, Package_SO:TSSOP-20_4.4x6.5mm_P0.65mm, symbol Audio:PCM5102A
Changed lines of the file:
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@@
-	)
-	(symbol
-		(lib_id "Audio:PCM5102A")
-		(at 137.16 144.78 0)
-		(unit 1)
-		(body_style 1)
-		(exclude_from_sim no)
-		(in_bom yes)
-		(on_board yes)
-		(in_pos_files yes)
-		(dnp no)
-		(fields_autoplaced yes)
-		(property "Reference" "U11"
-			(at 141.8433 127 0)
-			(show_name no)
-			(do_not_autoplace no)
-			(effects
-				(font
-					(size 1.27 1.27)
-				)
-				(justify left)
-			)
-		)
-		(property "Value" "PCM5102A"
-			(at 141.8433 129.54 0)
-			(show_name no)
-			(do_not_autoplace no)
-			(effects
-				(font
-					(size 1.27 1.27)
-				)
-				(justify left)
-			)
-		)
-		(property "Footprint" "Package_SO:TSSOP-20_4.4x6.5mm_P0.65mm"
-			(at 162.56 161.29 0)
-			(hide yes)
-			(show_name no)
-			(do_not_autoplace no)
-			(effects
-				(font
-					(size 1.27 1.27)
-				)
-			)
-		)
-		(property "Datasheet" "https://www.ti.com/lit/ds/symlink/pcm5102a.pdf"
-			(at 137.16 144.78 0)
-			(hide yes)
-			(show_name no)
-			(do_not_autoplace no)
-			(effects
-				(font
-					(size 1.27 1.27)
-				)
-			)
-		)
-		(property "Description" "2.1 VRMS, 112dB Audio Stereo DAC with PLL and 32-bit, 384kHz PCM Interface, TSSOP-20"
-			(at 137.16 144.78 0)
-			(hide yes)
-			(show_name no)
-			(do_not_autoplace no)
-			(effects
-				(font
-					(size 1.27 1.27)
-				)
-			)
-		)
-		(pin "15"
-		)
-		(pin "7"
-		)
-		(pin "5"
-		)
-		(pin "13"
-		)
-		(pin "17"
-		)
-		(pin "20"
-		)
-		(pin "8"
-		)
-		(pin "11"
-		)
-		(pin "16"
-		)
-		(pin "9"
-		)
-		(pin "12"
-		)
-		(pin "2"
-		)
-		(pin "18"
-		)
-		(pin "10"
-		)
-		(pin "3"
-		)
-		(pin "6"
-		)
-		(pin "14"
-		)
-		(pin "1"
-		)
-		(pin "19"
-		)
-		(pin "4"
-		)
-		(instances
-			(project "APM"
-				(path "/63e257c1-2fa4-4533-ab9e-932d24befb8c/298c3c38-2dcb-4443-81e3-86d0bc63c7e1"
-					(reference "U11")
-					(unit 1)
-				)
-			)
-		)
 	)
 	(symbol
