File: schematic/OSC_CTRL/OSC_CTRL/OSC_CTRL.kicad_sch (KiCad schematic)
At the start: 14 parts, among them SW1 SW_DIP_x08, SW2 SW_DIP_x08, U1 4052, U2 74AHC595

Commit message: wiring things up
Connections:
- net OSC1_WAVE1: now reaches U2.1 (QB)
- net OSC1_WAVE1: now also SW1.2
- net GPIO_595_SCLK: now reaches U2.11 (SRCLK)
- net GPIO_595_RCLK: now reaches U2.12 (RCLK)
- net GPIO_595_SER: now reaches U2.14 (SER)
- net OSC1_WAVE0: now reaches U2.15 (QA)
- net OSC1_WAVE0: now also SW1.1
- net OSC1_WAVE2: now reaches U2.2 (QC)
- net OSC1_WAVE2: now also SW1.3
- net OSC2_WAVE0: now reaches U2.3 (QD)
- net OSC2_WAVE0: now also SW2.1
- net OSC2_WAVE1: now reaches U2.4 (QE)
- net OSC2_WAVE1: now also SW2.2
- net OSC2_WAVE2: now reaches U2.5 (QF)
- net OSC2_WAVE2: now also SW2.3
