File: schematic/APM_v5_r1/APM.kicad_sch (KiCad schematic)
At the start: 25 parts, among them J10 Conn_02x17_Counter_Clockwise, J14 POT_FFC, J18 CTRL_FFC, J2 CAN, J4 LCD_display, J6 Conn_02x10_Counter_Clockwise, J8 Conn_02x15_Counter_Clockwise, J9 Conn_02x08_Counter_Clockwise

Commit message: getting the boards fabbed
Parts:
- added R49, R50: 2.2k, Resistor_SMD:R_0201_0603Metric, symbol Device:R
Connections:
- net 3V3_APM: now also R49.2, R50.2
- net APM_DBG_RX: now also U10.33 (PA10); no longer U10.25 (PB10)
- net APM_I2C2_SCL: now also R49.1
- net APM_I2C2_SDA: now also R50.1
- net APM_USER_RX: now reaches U10.18 (PB11)
- new net APM_USER_TX: U10.25 (PB10)
