File: schematic/APM_v5_r1/PMS_APM.kicad_sch (KiCad schematic)
At the start: 15 parts, among them U13 INA219AxD, U3 LT1963AxST-3.3, U7 INA219AxD

Commit message: getting the boards fabbed
Connections:
- net 3V3_LDO: now also C5.2, U13.5 (VS)
- net 5V_IN: no longer C5.2, U13.5 (VS)
Other:
- moved on the sheet: C5, C7, C9, D5, D7, R15, R16, R26, R28, R3, R30, R4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
