File: schematic/APM_v5_r1/STORAGE_APM.kicad_sch (KiCad schematic)
At the start: 16 parts, among them U4 W25Q128JVS, U5 MR25H40, U6 W25Q128JVS, U8 24LC1025-I_P

Commit message: getting the boards fabbed
Parts:
- JP3, JP4, JP5: now in the parts list
Changed lines of the file:
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@@
 		(body_style 1)
 		(exclude_from_sim no)
-		(in_bom no)
+		(in_bom yes)
 		(on_board yes)
 		(in_pos_files yes)
@@
 		(body_style 1)
 		(exclude_from_sim no)
-		(in_bom no)
+		(in_bom yes)
 		(on_board yes)
 		(in_pos_files yes)
@@
 		(body_style 1)
 		(exclude_from_sim no)
-		(in_bom no)
-		(on_board yes)
-		(in_pos_files yes)
+		(in_bom yes)
+		(on_board yes)
+		(in_pos_files yes)
