File: schematic/APM_v5_r2/APM.kicad_pcb (KiCad board)
At the start: 4 copper layers, 72.5 x 104.5 mm, 107 parts, among them J1 DF40C-60DS-0.4V(51), J11 DAC_L_PRB, J12 Conn_01x02, J14 ASDR_FFC, J16 USB_A_FEMALE, J18 WAVE_FFC, J19 AudioPlug3, J2 CAN, J23 VOL_L_CTRL, J24 VOL_R_CTRL, J3 DF40C-60DS-0.4V(51), J30 UART_DEBUG, J4 LCD_display, J5 Barrel_Jack, J7 DAC_R_PRB, U13 INA219AxD, U2 OPA1678, U3 LT1963AxST-3.3, U4 W25Q128JVS, U5 MR25H40, U6 W25Q128JVS, U7 INA219AxD, U8 24LC1025-I_P, U9 USBLC6-2SC6

Commit message: trying APM placement
Parts:
- removed J14: ASDR_FFC, Connector_FFC-FPC:Hirose_FH12-10S-0.5SH_1x10-1MP_P0.50mm_Horizontal
- removed J18: WAVE_FFC, Connector_FFC-FPC:Hirose_FH12-10S-0.5SH_1x10-1MP_P0.50mm_Horizontal
- added J6: OSC_CTRL, my_footprints:GCT_FFC2B28-20-G, B.Cu at (77.1, 105.1)
- added TP4: FPC_3V3_TP, TestPoint:TestPoint_Pad_D1.0mm, B.Cu at (79.5, 115.0)
- added TP9: FPC_GND_TP, TestPoint:TestPoint_Pad_D1.0mm, B.Cu at (76.7, 115.0)
- moved R91 101.4 mm to (75.2, 77.8)
- moved R92 101.0 mm to (75.2, 80.4)
- moved D63 100.0 mm to (72.8, 80.4), turned to 0 degrees
- moved D62 100.0 mm to (72.8, 77.8), turned to 0 degrees
- moved J30 99.7 mm to (78.1, 77.8)
- moved D19 84.6 mm to (78.1, 153.0), turned to 90 degrees
- moved R42 82.7 mm to (80.0, 152.2), turned to 0 degrees
- moved C17 42.5 mm to (72.1, 153.8)
- moved J4 42.5 mm to (72.1, 149.9)
- moved R50 37.0 mm to (131.1, 128.6), turned to 0 degrees
- moved R49 36.8 mm to (131.1, 126.1), turned to 0 degrees
Routing:
- net /APM_I2C2_SCL: track 0.00 -> 2.28 mm
- net /APM_I2C2_SDA: track 0.00 -> 2.28 mm

Commit message: renders. APM V5 R2 placement. going on with routing
Parts:
- removed J2: CAN, Connector_PinHeader_2.54mm:PinHeader_1x03_P2.54mm_Vertical
- R53, R7, R9: moved to B.Cu
- TP3, TP5, TP7: footprint TestPoint:TestPoint_Pad_1.5x1.5mm -> TestPoint:TestPoint_Pad_D1.0mm
- TP6, TP8: footprint TestPoint:TestPoint_Pad_1.5x1.5mm -> TestPoint:TestPoint_Pad_D1.0mm; moved to B.Cu
- moved R7 169.0 mm to (45.2, 103.4), turned to 180 degrees
- moved R53 169.0 mm to (45.2, 107.9), turned to 180 degrees
- moved R9 168.9 mm to (45.2, 112.5), turned to 180 degrees
- moved C2 129.8 mm to (84.0, 77.4)
- moved TP5 125.3 mm to (45.2, 101.7)
- moved TP7 125.2 mm to (45.2, 106.2)
- moved C15 124.8 mm to (90.5, 83.1)
- moved TP3 124.6 mm to (45.2, 110.8)
- moved C14 122.4 mm to (90.5, 88.0)
- moved U2 122.3 mm to (80.8, 85.6)
- moved C3 120.5 mm to (74.4, 81.9), turned to -90 degrees
- moved C12 117.4 mm to (77.1, 94.0), turned to -90 degrees
- moved C13 115.8 mm to (79.2, 94.0), turned to -90 degrees
- moved R46 113.1 mm to (77.1, 96.3)
- moved C10 111.3 mm to (82.4, 94.0), turned to -90 degrees
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Connections:
- R40 pad 2: /APM_LED_WARN -> /APM_LED_FAIL
- R41 pad 2: /APM_LED_FAIL -> /APM_LED_WARN
- U1 pad 13: /APM_LED_FAIL -> unconnected-(U1-PA13-Pad13)
- U1 pad 15: /APM_LED_OK -> unconnected-(U1-PA14-Pad15)
- U1 pad 17: /APM_LED_WARN -> unconnected-(U1-PA15-Pad17)
- U10 pad 13: /SR_GPIO1 -> /SEL_B_BIT_2
- U10 pad 15: /SR_GPIO2 -> /SEL_B_BIT_3
- U10 pad 16: unconnected-(U10-PB12-Pad16) -> /SEL_B_BIT_0
- U10 pad 17: unconnected-(U10-PB6-Pad17) -> /SEL_A_BIT_3
- U10 pad 24: unconnected-(U10-PB1-Pad24) -> /SEL_A_BIT_2
- U10 pad 27: unconnected-(U10-PB4-Pad27) -> /SEL_A_BIT_0
- U10 pad 29: unconnected-(U10-PB5-Pad29) -> /SEL_A_BIT_1
- U10 pad 60: unconnected-(U10-PF15-Pad60) -> /SEL_B_BIT_1
- U10 pad 64: unconnected-(U10-PE0-Pad64) -> /APM_LED_WARN
- U10 pad 66: unconnected-(U10-PG8-Pad66) -> /APM_LED_FAIL
- U10 pad 68: unconnected-(U10-PG5-Pad68) -> /APM_LED_OK
Routing:
- net 5V_APM: track 0.00 -> 101.8 mm, vias 0 -> 7
- net /DAC_1-1_R: track 0.00 -> 73.9 mm, vias 0 -> 1
- net /DAC_1-2_L: track 0.00 -> 64.1 mm, vias 0 -> 1
- net /MIDI_FS_D-: track 0.00 -> 57.9 mm
- net /MIDI_FS_D+: track 0.00 -> 56.8 mm
- net 3V3_APM: track 0.00 -> 37.3 mm, vias 0 -> 9
- net DAC_R_OUT: track 0.00 -> 27.5 mm
- net /APM_LED_WARN: track 0.00 -> 27.1 mm
- net 3V3_LDO: track 0.00 -> 24.8 mm, vias 0 -> 1
- net /APM_LED_FAIL: track 0.00 -> 22.9 mm
- net DAC_L_OUT: track 0.00 -> 19.5 mm
- net /APM_LED_OK: track 0.00 -> 18.2 mm
- net /APM_I2C2_SDA: track 2.28 -> 19.0 mm, vias 0 -> 1
- net /APM_I2C2_SCL: track 2.28 -> 18.6 mm, vias 0 -> 1
- net Net-(U2A-+): track 0.00 -> 13.3 mm
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- added copper zone on B.Cu, net /PMS_APM/5V_PWR_IN
- added copper zone on In1.Cu, net 3V3_APM
- added copper zone on B.Cu, net 3V3_LDO
- added copper zone on B.Cu, net 5V_APM
- removed copper zone on In1.Cu, net 5V_APM
Other:
- board text added: "3v3 LDO"
- board text added: "5V IN"
- board text added: "ACM_PWR"
- board text added: "APM_PWR"
- board text added: "AUDIO OUT"
- board text added: "FAIL"
- board text added: "L"
- board text added: "MIDI IN"
- board text added: "MIDI_D+"
- board text added: "MIDI_D-"
- board text added: "OK"
- board text added: "OUT"
- board text added: "R"
- board text added: "RXD"
- board text added: "TXD"
- board text added: "VOL"
- board text added: "WARN"
- board text removed: "PWR_IN"

Commit message: autorouter thingy working decent? most of the 60P connectors routed? i should verify dimentions first
Routing:
- net /APM_FMC_NWAIT: track 0.00 -> 99.9 mm, vias 0 -> 1
- net /APM_FMC_DA13: track 0.00 -> 92.2 mm, vias 0 -> 1
- net /APM_I2C2_SCL: track 18.6 -> 91.2 mm, vias 1 -> 5
- net /QSPI1_NCS: track 0.00 -> 72.1 mm
- net /APM_I2C2_SDA: track 19.0 -> 90.9 mm, vias 1 -> 5
- net /APM_SPI1_SCK: track 0.00 -> 69.5 mm, vias 0 -> 4
- net /APM_SPI1_MISO: track 0.00 -> 68.6 mm, vias 0 -> 2
- net /QSPI1_D0: track 0.00 -> 67.5 mm, vias 0 -> 2
- net /APM_FMC_NE1: track 0.00 -> 63.6 mm, vias 0 -> 2
- net /APM_SPI1_MOSI: track 0.00 -> 62.8 mm, vias 0 -> 2
- net /APM_FPGA_UART_RX: track 0.00 -> 58.9 mm, vias 0 -> 2
- net /QSPI1_D1: track 0.00 -> 50.4 mm, vias 0 -> 1
- net /APM_FPGA_UART_TX: track 0.00 -> 49.7 mm, vias 0 -> 2
- net /QSPI_SCK2: track 0.00 -> 49.2 mm, vias 0 -> 1
- net /APM_FMC_CLK: track 0.00 -> 48.4 mm, vias 0 -> 1
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
Commit message: fills
Routing:
- net GND: vias 4 -> 8
Other:
- board text added: "mid conn to mid conn is 11.2mm"
Changed lines of the file:
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@@
 		)
 	)
+	(gr_text "mid conn to mid conn is 11.2mm"
+		(at 103.2 150.6 0)
+		(layer "B.SilkS")
+		(effects
+			(font
+				(size 0.6 0.6)
+				(thickness 0.1)
+				(bold yes)
+			)
+			(justify left bottom mirror)
+		)
+	)
 	(gr_text "MIDI IN"
 		(locked yes)
@@
 	)
 	(via
+		(at 82.3 138.1)
+		(size 0.5)
+		(drill 0.3)
+		(layers "F.Cu" "B.Cu")
+		(free yes)
+		(net "GND")
+	)
+	(via
 		(at 122.85 128.5)
 		(size 0.5)
@@
 	)
 	(via
+		(at 79.7 139.4)
+		(size 0.5)
+		(drill 0.3)
+		(layers "F.Cu" "B.Cu")
+		(free yes)
+		(net "GND")
+	)
+	(via
+		(at 92 140.2)
+		(size 0.5)
+		(drill 0.3)
+		(layers "F.Cu" "B.Cu")
+		(free yes)
+		(net "GND")
+	)
+	(via
+		(at 92.6 142.1)
+		(size 0.5)
+		(drill 0.3)
+		(layers "F.Cu" "B.Cu")
+		(free yes)
+		(net "GND")
+	)
+	(via
 		(at 113 113.295)
 		(size 0.3)
@@
 		(members "1887b254-e2ed-4d87-8881-0635cb73fef5" "62be610a-afe6-4010-909d-777f08e645da"
 			"6ed8da5a-25e4-41bf-929f-2daf9c413d9b" "741fe7ab-0478-4c5c-9463-7179d6dfa343"
-			"79a344b1-a80d-492a-96fc-1fb1ef97a04b" "a4e288e5-5c9e-461a-a69b-f9016030adf2"
-			"b9769bae-ff1d-4018-bf9c-5ef7fbd0519e" "cd4a51cb-1577-4c6b-8eda-b60fa1f357c2"
-			"d49c1673-6689-4437-befe-82b0b7b1550e" "de62111a-03d5-4f33-9e8b-468bec9e5041"
+			"79a344b1-a80d-492a-96fc-1fb1ef97a04b"
 		)
 	)

Commit message: routed and passing DRC except for the differentials for USB
Parts:
- J30: footprint Connector_PinHeader_2.54mm:PinHeader_1x03_P2.54mm_Vertical -> Connector_PinHeader_2.54mm:PinHeader_1x03_P2.54mm_Vertical_SMD_Pin1Left
- J4: footprint Connector_PinHeader_2.54mm:PinHeader_1x04_P2.54mm_Vertical -> Connector_PinHeader_2.54mm:PinHeader_1x04_P2.54mm_Vertical_SMD_Pin1Left
- moved J4 57.9 mm to (107.7, 91.7)
- moved C17 56.2 mm to (106.0, 98.4), turned to 0 degrees
- moved R7 55.1 mm to (96.9, 84.4)
- moved TH2 55.1 mm to (101.8, 83.5)
- moved TP5 55.1 mm to (96.9, 82.7)
- moved J30 50.8 mm to (78.4, 125.4)
- moved D62 48.0 mm to (71.8, 122.8)
- moved D63 48.0 mm to (71.7, 125.4)
- moved R92 48.0 mm to (74.2, 125.4)
- moved R91 48.0 mm to (74.2, 122.8)
- moved R53 41.8 mm to (70.8, 74.9)
- moved TH4 41.8 mm to (75.6, 74.0)
- moved TP7 41.8 mm to (70.8, 73.2)
- moved R9 30.7 mm to (75.2, 118.9)
- moved TH5 30.7 mm to (80.0, 118.1)
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Routing:
- net 5V_APM: track 101.8 -> 208.1 mm, vias 7 -> 8
- net /APM_FMC_NL: track 0.00 -> 84.9 mm, vias 0 -> 2
- net /APM_DBG_TX: track 2.54 -> 44.1 mm, vias 0 -> 2
- net /APM_DBG_RX: track 2.57 -> 32.8 mm, vias 0 -> 1
- net /APM_SPI1_CS: track 0.00 -> 25.1 mm, vias 0 -> 1
- net /APM_SPI1_SCK: track 69.5 -> 90.0 mm
- net /APM_I2C2_SCL: track 91.2 -> 110.8 mm, vias 5 -> 6
- net /APM_I2C2_SDA: track 90.9 -> 100.1 mm
- net /APM_FMC_NWAIT: track 99.9 -> 108.4 mm
- net 3V3_APM: track 63.6 -> 59.4 mm, vias 16 -> 15
- net /APM_FMC_DA1: track 48.3 -> 51.9 mm
- net /APM_FMC_DA6: track 46.3 -> 48.7 mm
- net Net-(R7-Pad1): track 0.00 -> 2.33 mm
- net Net-(R53-Pad1): track 0.00 -> 2.31 mm
- net Net-(R9-Pad1): track 0.00 -> 2.30 mm
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