File: schematic/APM_v5_r2/FPGA_INTERFACE.kicad_sch (KiCad schematic)
At the start: 6 parts, among them J1 DF40C-60DS-0.4V(51), J15 FPGA FFC, J21 FPGA FMC, J3 DF40C-60DS-0.4V(51)

Commit message: fixed ACM A19 not routed
Connections:
- net FPGA_I2C2_SCL: now also J1.34 (Pin_34); no longer J1.32 (Pin_32)
- net FPGA_I2C2_SDA: now also J1.32 (Pin_32); no longer J1.30 (Pin_30)
