File: schematic/APM_v5_r2/PMS_APM.kicad_sch (KiCad schematic)
At the start: 15 parts, among them U13 INA219AxD, U3 LT1963AxST-3.3, U7 INA219AxD

Commit message: adding new rev of apm board with new routing and power management
Parts:
- added C18: 220uF 10V, Capacitor_SMD:CP_Elec_4x3, symbol Device:C_Small
- added D2: 20V 3A, Diode_SMD:D_SOD-123, symbol Device:D_Schottky
- added D3: SMAJ5.0A, Diode_SMD:D_SMA, symbol Device:D_Schottky
- added D6: RED_LED_PWR, LED_SMD:LED_0603_1608Metric, symbol Device:LED
- added F1: 6V 2A, Fuse:Fuse_0603_1608Metric, symbol Device:Polyfuse_Small
- added J5: Barrel_Jack, Connector_BarrelJack:BarrelJack_GCT_DCJ200-10-A_Horizontal, symbol Connector:Barrel_Jack
- added R19: 4.7k, Resistor_SMD:R_0201_0603Metric, symbol Device:R
Connections:
- net GND: now also C18.2, D2.2 (A), D3.2 (A), D6.1 (K), J5.2
- net 5V_IN renamed 5V_PWR_IN
- net 5V_PWR_IN: now also C18.1, D2.1 (K), D3.1 (K), F1.1, R19.2
- new net: F1.2, J5.1
- new net: D6.2 (A), R19.1
Other:
- note added: "Barrel Jack connector provides 5V to the board"
- note added: "POWER INPUT"
- moved on the sheet: C5, C7, C9, D5, D7, R15, R16, R26, R28, R3, R30, R4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
