File: schematic/ACM_v1_r1/ACM_v1_r1.kicad_pcb (KiCad board)
At the start: 4 copper layers, 25.5 x 39.9 mm, 38 parts, among them J1 DF40C-60DS-0.4V(51), J2 DF40C-60DS-0.4V(51), J3 Conn_02x04_Odd_Even, J4 Conn_01x02, J5 DF40C-60DS-0.4V(51), J6 DF40C-60DS-0.4V(51), SW1 RST

Commit message: fixed ACM A19 not routed
Parts:
- moved G*** 5.97 mm to (142.0, 121.2)
Connections:
- J6 pad 22: unconnected-(J6-Pin_22-Pad22) -> /L4_IOR31A_40P
Routing:
- net /L4_IOR31A_40P: track 0.00 -> 1.66 mm, vias 0 -> 1
Changed lines of the file:
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@@
 			(layers "B.Cu" "B.Mask" "B.Paste")
 			(roundrect_rratio 0.25)
-			(net "unconnected-(J6-Pin_22-Pad22)")
+			(net "/L4_IOR31A_40P")
 			(pinfunction "Pin_22_22")
 			(pintype "passive")
@@
 	(footprint "graphics:obese_bulldog_15x16mm"
 		(layer "B.Cu")
-		(at 141.473938 115.202421 -90)
+		(at 141.983938 121.152421 -90)
 		(property "Reference" "G***"
 			(at 0 0 90)
@@
 	)
 	(segment
+		(start 148.24 99.68)
+		(end 149.07 99.68)
+		(width 0.1)
+		(layer "F.Cu")
+		(net "/L4_IOR31A_40P")
+	)
+	(via
+		(at 149.07 99.68)
+		(size 0.3)
+		(drill 0.2)
+		(layers "F.Cu" "B.Cu")
+		(net "/L4_IOR31A_40P")
+	)
+	(segment
+		(start 148.24 99.68)
+		(end 149.07 99.68)
+		(width 0.1)
+		(layer "B.Cu")
+		(net "/L4_IOR31A_40P")
+	)
+	(segment
