File: schematic/AUDIO_BOARD_v1_r1/AUDIO_BOARD.kicad_sch (KiCad schematic)
At the start: 38 parts, among them J1 PWR FFC 4p, J2 U.FL L in, J3 U.FL R in, J4 1/4in L, J5 1/4in R, J6 3.5mm HP, U1 ICL7660, U2 OPA1678, U3 OPA1678

Commit message: audio master board
Parts:
- added RV4, RV5: VOL 10k (dual-gang), symbol Device:R_Potentiometer
- added RV6: R_Potentiometer_Dual, symbol Device:R_Potentiometer_Dual
Connections:
- net FILT_L_OUT: now also RV4.1; no longer J4.T1, R9.1
- net FILT_R_OUT: now also RV5.1; no longer J5.T1, R10.1
- net GND: now also RV4.3, RV5.3
- net at C11.2, U2.5 (+): now also C12.1, R6.2
- net at C8.1, R3.2: now also C7.2, U2.3 (+); no longer R2.2
- net at R6.1: now also R5.2
- net at R3.1: now also R2.2
- new net VOL_L: J4.T1, R9.1, RV4.2
- new net VOL_R: J5.T1, R10.1, RV5.2
Other:
- note added: "AUDIO INPUT - U.FL for L and R DACs from APM"
- note added: "MASTER VOLUME - RV4/RV5 = one dual-gang pot (shared L/R knob); attenuates final output to the jacks/HP"
- moved on the sheet: C18, C19, C20, C21, R3, R6

Commit message: osc ctrl has black mask, sent to JLCPCB. APM routed. also sent to JLCPCB.figuring out the master audio control board
Parts:
- added C60: 1uF, Capacitor_SMD:C_0805_2012Metric, symbol Device:C_Small
- added C61: 22uF, Capacitor_SMD:C_0805_2012Metric, symbol Device:C_Small
- added U15: LTC660, Package_SO:SOIC-8_3.9x4.9mm_P1.27mm, symbol Regulator_SwitchedCapacitor:LTC660
- U1: value ICL7660 -> LTC660; symbol Regulator_SwitchedCapacitor:ICL7660 -> Regulator_SwitchedCapacitor:LTC660
Connections:
- net +5V: now also U1.1 (BOOST), U15.1 (BOOST), U15.8 (V+)
- net -5V: now also C61.1, U15.5 (VOUT)
- net FILT_L_OUT: no longer RV4.1
- net FILT_R_OUT: no longer RV5.1
- net GND: now also C61.2, U15.3 (GND)
- new net: C60.1, U15.2 (CAP+)
- new net: C60.2, U15.4 (CAP-)
- new net FX_L_OUT: RV4.1
- new net FX_R_OUT: RV5.1
Other:
- added sheet FX_CHAIN (FX_CHAIN.kicad_sch)
- added sheet FX_CONTROL (FX_CONTROL.kicad_sch)
- added sheet MASTER_FILTER (MASTER_FILTER.kicad_sch)

Commit message: working on chorus and phaser
Parts:
- removed RV4, RV5: VOL 10k (dual-gang), symbol Device:R_Potentiometer
- removed RV6: R_Potentiometer_Dual, symbol Device:R_Potentiometer_Dual
Connections:
- net VOL_L is gone; now on net FX_L_OUT: J4.T1, R9.1
- net VOL_R is gone; now on net FX_L_OUT: J5.T1, R10.1
- net -5V: now also C11.1, C7.1
- net FX_L_OUT: now also C16.2, C17.2, J6.R, J6.T
- net GND: now also C11.2, C12.1, C7.2, C8.1, R3.2, R6.2, U2.3 (+), U2.5 (+)
- no-connect marks 0 -> 12
Other:
- sheet MASTER_FILTER ports: added none; removed ORDER_SEL
- moved on the sheet: C11, C12, C13, C18, C19, C20, C21, C6, C60, C61, C7, C8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

Commit message: phaser? schematic is messy
Parts:
- added J1: PWR FFC, Connector_FFC-FPC:Amphenol_F32Q-1A7x1-11004_1x04-1MP_P0.5mm_Horizontal, symbol Connector_Generic:Conn_01x04
- added J7: CTRL FFC, Connector_FFC-FPC:Amphenol_F32Q-1A7x1-11010_1x10-1MP_P0.5mm_Horizontal, symbol Connector_Generic:Conn_01x10
Connections:
- net +5V: now also J1.1 (Pin_1)
- net FX_L_OUT: no longer C16.2, C17.2, J4.T1, J5.T1, J6.R, J6.T, R10.1, R9.1
- net GND: now also J1.3 (Pin_3), J1.4 (Pin_4), J7.8 (Pin_8), J7.9 (Pin_9)
- new net +3V3: J1.2 (Pin_2)
- new net CS_DAC1: J7.4 (Pin_4)
- new net CS_DAC2: J7.5 (Pin_5)
- new net CS_EXP: J7.6 (Pin_6)
- new net SPI_MISO: J7.3 (Pin_3)
- new net SPI_MOSI: J7.2 (Pin_2)
- new net SPI_SCK: J7.1 (Pin_1)
- new net VOL_L: C16.2, C17.2, J4.T1, J5.T1, J6.R, J6.T, R10.1, R9.1
- no-connect marks 12 -> 14
Other:
- added sheet FX_CHORUS (FX_CHORUS.kicad_sch)
- added sheet FX_PHASER (FX_PHASER.kicad_sch)
- sheet ANALOG_FILTER_CV ports: added CS_DAC1, CV_FX3, MODE_SEL, SPI_MOSI, SPI_SCK; removed none
- sheet FX_CONTROL ports: added CS_DAC2, CS_EXP, FX_EN3, GATE, MODE_SEL, SPI_MISO, SPI_MOSI, SPI_SCK; removed none
- note added: "CONTROL FFC (10-pin from APM J8): 1SCK 2MOSI 3MISO 4CS_DAC1 5CS_DAC2 6CS_EXP 7sp 8/9GND 10sp"
- note added: "POWER FFC (4-pin from APM): +5V +3V3 GND GND (-5V made on-board)"

Commit message: LDO?
Parts:
- removed J1: PWR FFC, Connector_FFC-FPC:Amphenol_F32Q-1A7x1-11004_1x04-1MP_P0.5mm_Horizontal, symbol Connector_Generic:Conn_01x04
