File: schematic/AUDIO_BOARD_v1_r1/FX_CONTROL.kicad_sch (KiCad schematic)
At the start: 6 parts, among them J20 FX-CTRL FFC, U20 DAC8565

Commit message: phaser? schematic is messy
Parts:
- removed J20: FX-CTRL FFC, Connector_FFC-FPC:Amphenol_F32Q-1A7x1-11010_1x10-1MP_P0.5mm_Horizontal, symbol Connector_Generic:Conn_01x10
- added C55: 100nF, Capacitor_SMD:C_0402_1005Metric, symbol Device:C_Small
- added U21: MCP23S17, Package_SO:SOIC-28W_7.5x17.9mm_P1.27mm, symbol Custom:MCP23S17
Connections:
- net FX_EN1: now also U21.21 (GPA0)
- net FX_EN2: now also U21.22 (GPA1)
- net GND: now also C55.2, U21.10 (VSS), U21.15 (A0), U21.16 (A1), U21.17 (A2)
- net MODE_A: now also U21.24 (GPA3)
- net MODE_B: now also U21.25 (GPA4)
- net ORDER_SEL: now also U21.26 (GPA5)
- net SPI_MOSI2 renamed SPI_MOSI
- net SPI_MOSI: now also U21.13 (SI)
- net SPI_SCK2 renamed SPI_SCK
- net SPI_SCK: now also U21.12 (SCK)
- new net +3V3: C55.1, U21.18 (~{RESET}), U21.9 (VDD)
- new net CS_EXP: U21.11 (~{CS})
- new net FX_EN3: U21.23 (GPA2)
- new net GATE: U21.27 (GPA6)
- new net MODE_SEL: U21.28 (GPA7)
- new net SPI_MISO: U21.14 (SO)
- no-connect marks 0 -> 10
Other:
- note added: "CONTROL - SPI + CS_DAC2 + CS_EXP come from the root's one 10-pin control FFC. This DAC + the MCP expander sit on that shared SPI bus."
- note added: "MCP23S17 expander - SPI2 + CS_EXP -> 16 GPIO fan-out for all FX/filter digital selects (frees the FFC from per-line GPIO). Runs at +3V3."
- note removed: "FX-CTRL FFC: 1SCK 2MOSI 3CS_DAC2 4MODE_A 5MODE_B 6ORDER_SEL 7FX_EN1 8FX_EN2 9/10GND"

Commit message: sim, render, audio stuff
Other:
- note added: "CONTROL/DAC - SPI + CS_DAC2 + CS_EXP from the root's one 10-pin control FFC; this DAC + the MCP expander share that SPI bus."
- note removed: "CONTROL - SPI + CS_DAC2 + CS_EXP come from the root's one 10-pin control FFC. This DAC + the MCP expander sit on that shared SPI bus."
- note removed: "DAC8565 #2 - 4 CV channels for the master filter/FX"
Changed lines of the file:
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@@
 	(text "FX CONTROL  -  2nd FX-control FFC (SPI + mode/order/enable) -> DAC8565 #2 makes CV_CUTOFF/CV_RES (+2 spare FX CVs); digital selects pass through" (exclude_from_sim no) (at 16 15 0) (effects (font (size 1.9 1.9) ) (justify left bottom)))
 	(text "Knobs/switches live on the controller board; STM32 reads them, drives this DAC over SPI and sets the digital lines." (exclude_from_sim no) (at 16 250 0) (effects (font (size 1.5 1.5) ) (justify left bottom)))
-	(text "CONTROL  -  SPI + CS_DAC2 + CS_EXP come from the root's one 10-pin control FFC. This DAC + the MCP expander sit on that shared SPI bus." (exclude_from_sim no) (at 16 30 0) (effects (font (size 1.5 1.5) ) (justify left bottom)))
-	(hierarchical_label "SPI_SCK" (shape input) (at 30.48 39.37 0) (effects (font (size 1.27 1.27)) (justify left)))
-	(label "SPI_SCK" (at 30.48 39.37 0) (effects (font (size 1.27 1.27)) (justify left bottom)))
-	(hierarchical_label "SPI_MOSI" (shape input) (at 30.48 45.72 0) (effects (font (size 1.27 1.27)) (justify left)))
-	(label "SPI_MOSI" (at 30.48 45.72 0) (effects (font (size 1.27 1.27)) (justify left bottom)))
-	(hierarchical_label "SPI_MISO" (shape input) (at 30.48 52.07 0) (effects (font (size 1.27 1.27)) (justify left)))
-	(label "SPI_MISO" (at 30.48 52.07 0) (effects (font (size 1.27 1.27)) (justify left bottom)))
-	(hierarchical_label "CS_DAC2" (shape input) (at 30.48 58.42 0) (effects (font (size 1.27 1.27)) (justify left)))
-	(label "CS_DAC2" (at 30.48 58.42 0) (effects (font (size 1.27 1.27)) (justify left bottom)))
-	(hierarchical_label "CS_EXP" (shape input) (at 30.48 63.5 0) (effects (font (size 1.27 1.27)) (justify left)))
-	(label "CS_EXP" (at 30.48 63.5 0) (effects (font (size 1.27 1.27)) (justify left bottom)))
-	(text "DAC8565 #2  -  4 CV channels for the master filter/FX" (exclude_from_sim no) (at 100 30 0) (effects (font (size 1.6 1.6) ) (justify left bottom)))
+	(text "CONTROL/DAC  -  SPI + CS_DAC2 + CS_EXP from the root's one 10-pin control FFC; this DAC + the MCP expander share that SPI bus." (exclude_from_sim no) (at 16 30 0) (effects (font (size 1.5 1.5) ) (justify left bottom)))
 	(symbol (lib_id "Analog_DAC:DAC8565") (at 119.38 69.85 0) (unit 1)
 		(exclude_from_sim no) (in_bom yes) (on_board yes) (dnp no)
@@
 		(instances (project "AUDIO_BOARD" (path "/ba93534c-f2e3-4dc0-9a76-585fdc68cf39/c0ffee00-1111-2222-3333-444455556666" (reference "U20") (unit 1)))))
 	(wire (pts (xy 106.68 62.23) (xy 95.25 62.23)) (stroke (width 0) (type default)))
-	(label "SPI_SCK" (at 95.25 62.23 0) (effects (font (size 1.27 1.27)) (justify left bottom)))
+	(hierarchical_label "SPI_SCK" (shape input) (at 95.25 62.23 0) (effects (font (size 1.27 1.27)) (justify left)))
 	(wire (pts (xy 106.68 64.77) (xy 95.25 64.77)) (stroke (width 0) (type default)))
-	(label "SPI_MOSI" (at 95.25 64.77 0) (effects (font (size 1.27 1.27)) (justify left bottom)))
+	(hierarchical_label "SPI_MOSI" (shape input) (at 95.25 64.77 0) (effects (font (size 1.27 1.27)) (justify left)))
 	(wire (pts (xy 106.68 59.69) (xy 95.25 59.69)) (stroke (width 0) (type default)))
-	(label "CS_DAC2" (at 95.25 59.69 0) (effects (font (size 1.27 1.27)) (justify left bottom)))
+	(hierarchical_label "CS_DAC2" (shape input) (at 95.25 59.69 0) (effects (font (size 1.27 1.27)) (justify left)))
 	(wire (pts (xy 106.68 57.15) (xy 99.06 57.15)) (stroke (width 0) (type default)))
 	(symbol (lib_id "power:GND") (at 99.06 57.15 0) (unit 1)
@@
 		(instances (project "AUDIO_BOARD" (path "/ba93534c-f2e3-4dc0-9a76-585fdc68cf39/c0ffee00-1111-2222-3333-444455556666" (reference "#PWR417") (unit 1)))))
 	(wire (pts (xy 109.22 170.18) (xy 101.6 170.18)) (stroke (width 0) (type default)))
-	(label "CS_EXP" (at 101.6 170.18 0) (effects (font (size 1.27 1.27)) (justify left bottom)))
+	(hierarchical_label "CS_EXP" (shape input) (at 101.6 170.18 0) (effects (font (size 1.27 1.27)) (justify left)))
 	(wire (pts (xy 109.22 172.72) (xy 101.6 172.72)) (stroke (width 0) (type default)))
 	(label "SPI_SCK" (at 101.6 172.72 0) (effects (font (size 1.27 1.27)) (justify left bottom)))
@@
 	(label "SPI_MOSI" (at 101.6 175.26 0) (effects (font (size 1.27 1.27)) (justify left bottom)))
 	(wire (pts (xy 109.22 177.8) (xy 101.6 177.8)) (stroke (width 0) (type default)))
-	(label "SPI_MISO" (at 101.6 177.8 0) (effects (font (size 1.27 1.27)) (justify left bottom)))
+	(hierarchical_label "SPI_MISO" (shape input) (at 101.6 177.8 0) (effects (font (size 1.27 1.27)) (justify left)))
 	(wire (pts (xy 109.22 187.96) (xy 101.6 187.96)) (stroke (width 0) (type default)))
 	(symbol (lib_id "power:+3V3") (at 101.6 187.96 0) (unit 1)

Commit message: LDO?
Parts:
- added C56, C57: 1uF, Capacitor_SMD:C_0402_1005Metric, symbol Device:C_Small
- added U22: AP2112K-3.3, Package_TO_SOT_SMD:SOT-23-5, symbol Regulator_Linear:AP2112K-3.3
Connections:
- net +3V3: now also C57.1, U22.5 (VOUT)
- net +5V: now also C56.1, U22.1 (VIN), U22.3 (EN)
- net GND: now also C56.2, C57.2, U22.2 (GND)
- no-connect marks 10 -> 11
Other:
- note added: "+3V3 LDO - AP2112K-3.3 from +5V (power FFC carries no +3V3); supplies only the MCP expander."
Changed lines of the file:
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@@
 		(instances (project "AUDIO_BOARD" (path "/ba93534c-f2e3-4dc0-9a76-585fdc68cf39/c0ffee00-1111-2222-3333-444455556666" (reference "#PWR423") (unit 1)))))
 	(wire (pts (xy 96.52 187.96) (xy 96.52 191.77)) (stroke (width 0) (type default)))
-	(symbol (lib_id "power:PWR_FLAG") (at 76.2 39.37 0) (unit 1)
+	(text "+3V3 LDO  -  AP2112K-3.3 from +5V (power FFC carries no +3V3); supplies only the MCP expander." (exclude_from_sim no) (at 16 192 0) (effects (font (size 1.4 1.4) ) (justify left bottom)))
+	(symbol (lib_id "Regulator_Linear:AP2112K-3.3") (at 39.37 199.39 0) (unit 1)
 		(exclude_from_sim no) (in_bom yes) (on_board yes) (dnp no)
-		(property "Reference" "#FLG424" (at 76.2 36.37 0) (effects (font (size 1.27 1.27)) (hide yes)))
-		(property "Value" "PWR_FLAG" (at 76.2 41.87 0) (effects (font (size 1.27 1.27))))
-		(instances (project "AUDIO_BOARD" (path "/ba93534c-f2e3-4dc0-9a76-585fdc68cf39/c0ffee00-1111-2222-3333-444455556666" (reference "#FLG424") (unit 1)))))
-	(wire (pts (xy 76.2 39.37) (xy 76.2 36.83)) (stroke (width 0) (type default)))
-	(symbol (lib_id "power:+3V3") (at 76.2 36.83 0) (unit 1)
+		(property "Reference" "U22" (at 41.37 197.39 0) (effects (font (size 1.27 1.27)) (justify left)))
+		(property "Value" "AP2112K-3.3" (at 41.37 201.39 0) (effects (font (size 1.27 1.27)) (justify left)))
+		(property "Footprint" "Package_TO_SOT_SMD:SOT-23-5" (at 39.37 199.39 0) (effects (font (size 1.27 1.27)) (hide yes)))
+		(instances (project "AUDIO_BOARD" (path "/ba93534c-f2e3-4dc0-9a76-585fdc68cf39/c0ffee00-1111-2222-3333-444455556666" (reference "U22") (unit 1)))))
+	(wire (pts (xy 31.75 196.85) (xy 25.4 196.85)) (stroke (width 0) (type default)))
+	(symbol (lib_id "power:+5V") (at 25.4 196.85 0) (unit 1)
 		(exclude_from_sim no) (in_bom yes) (on_board yes) (dnp no)
-		(property "Reference" "#PWR425" (at 76.2 39.83 0) (effects (font (size 1.27 1.27)) (hide yes)))
-		(property "Value" "+3V3" (at 76.2 33.83 0) (effects (font (size 1.27 1.27))))
+		(property "Reference" "#PWR424" (at 25.4 199.85 0) (effects (font (size 1.27 1.27)) (hide yes)))
+		(property "Value" "+5V" (at 25.4 193.85 0) (effects (font (size 1.27 1.27))))
+		(instances (project "AUDIO_BOARD" (path "/ba93534c-f2e3-4dc0-9a76-585fdc68cf39/c0ffee00-1111-2222-3333-444455556666" (reference "#PWR424") (unit 1)))))
+	(wire (pts (xy 31.75 199.39) (xy 25.4 199.39)) (stroke (width 0) (type default)))
+	(symbol (lib_id "power:+5V") (at 25.4 199.39 0) (unit 1)
+		(exclude_from_sim no) (in_bom yes) (on_board yes) (dnp no)
+		(property "Reference" "#PWR425" (at 25.4 202.39 0) (effects (font (size 1.27 1.27)) (hide yes)))
+		(property "Value" "+5V" (at 25.4 196.39 0) (effects (font (size 1.27 1.27))))
 		(instances (project "AUDIO_BOARD" (path "/ba93534c-f2e3-4dc0-9a76-585fdc68cf39/c0ffee00-1111-2222-3333-444455556666" (reference "#PWR425") (unit 1)))))
+	(wire (pts (xy 39.37 207.01) (xy 39.37 210.82)) (stroke (width 0) (type default)))
+	(symbol (lib_id "power:GND") (at 39.37 210.82 0) (unit 1)
+		(exclude_from_sim no) (in_bom yes) (on_board yes) (dnp no)
+		(property "Reference" "#PWR426" (at 39.37 213.82 0) (effects (font (size 1.27 1.27)) (hide yes)))
+		(property "Value" "GND" (at 39.37 207.82 0) (effects (font (size 1.27 1.27))))
+		(instances (project "AUDIO_BOARD" (path "/ba93534c-f2e3-4dc0-9a76-585fdc68cf39/c0ffee00-1111-2222-3333-444455556666" (reference "#PWR426") (unit 1)))))
+	(no_connect (at 44.45 199.39))
+	(wire (pts (xy 46.99 196.85) (xy 53.34 196.85)) (stroke (width 0) (type default)))
+	(symbol (lib_id "power:+3V3") (at 53.34 196.85 0) (unit 1)
+		(exclude_from_sim no) (in_bom yes) (on_board yes) (dnp no)
+		(property "Reference" "#PWR427" (at 53.34 199.85 0) (effects (font (size 1.27 1.27)) (hide yes)))
+		(property "Value" "+3V3" (at 53.34 193.85 0) (effects (font (size 1.27 1.27))))
+		(instances (project "AUDIO_BOARD" (path "/ba93534c-f2e3-4dc0-9a76-585fdc68cf39/c0ffee00-1111-2222-3333-444455556666" (reference "#PWR427") (unit 1)))))
+	(symbol (lib_id "Device:C_Small") (at 21.59 205.74 0) (unit 1)
+		(exclude_from_sim no) (in_bom yes) (on_board yes) (dnp no)
+		(property "Reference" "C56" (at 23.59 203.74 0) (effects (font (size 1.27 1.27)) (justify left)))
+		(property "Value" "1uF" (at 23.59 207.74 0) (effects (font (size 1.27 1.27)) (justify left)))
+		(property "Footprint" "Capacitor_SMD:C_0402_1005Metric" (at 21.59 205.74 0) (effects (font (size 1.27 1.27)) (hide yes)))
+		(instances (project "AUDIO_BOARD" (path "/ba93534c-f2e3-4dc0-9a76-585fdc68cf39/c0ffee00-1111-2222-3333-444455556666" (reference "C56") (unit 1)))))
+	(symbol (lib_id "power:+5V") (at 21.59 199.39 0) (unit 1)
+		(exclude_from_sim no) (in_bom yes) (on_board yes) (dnp no)
+		(property "Reference" "#PWR428" (at 21.59 202.39 0) (effects (font (size 1.27 1.27)) (hide yes)))
+		(property "Value" "+5V" (at 21.59 196.39 0) (effects (font (size 1.27 1.27))))
+		(instances (project "AUDIO_BOARD" (path "/ba93534c-f2e3-4dc0-9a76-585fdc68cf39/c0ffee00-1111-2222-3333-444455556666" (reference "#PWR428") (unit 1)))))
+	(wire (pts (xy 21.59 203.2) (xy 21.59 199.39)) (stroke (width 0) (type default)))
+	(symbol (lib_id "power:GND") (at 21.59 212.09 0) (unit 1)
+		(exclude_from_sim no) (in_bom yes) (on_board yes) (dnp no)
+		(property "Reference" "#PWR429" (at 21.59 215.09 0) (effects (font (size 1.27 1.27)) (hide yes)))
+		(property "Value" "GND" (at 21.59 209.09 0) (effects (font (size 1.27 1.27))))
+		(instances (project "AUDIO_BOARD" (path "/ba93534c-f2e3-4dc0-9a76-585fdc68cf39/c0ffee00-1111-2222-3333-444455556666" (reference "#PWR429") (unit 1)))))
+	(wire (pts (xy 21.59 208.28) (xy 21.59 212.09)) (stroke (width 0) (type default)))
+	(symbol (lib_id "Device:C_Small") (at 58.42 205.74 0) (unit 1)
+		(exclude_from_sim no) (in_bom yes) (on_board yes) (dnp no)
+		(property "Reference" "C57" (at 60.42 203.74 0) (effects (font (size 1.27 1.27)) (justify left)))
+		(property "Value" "1uF" (at 60.42 207.74 0) (effects (font (size 1.27 1.27)) (justify left)))
+		(property "Footprint" "Capacitor_SMD:C_0402_1005Metric" (at 58.42 205.74 0) (effects (font (size 1.27 1.27)) (hide yes)))
+		(instances (project "AUDIO_BOARD" (path "/ba93534c-f2e3-4dc0-9a76-585fdc68cf39/c0ffee00-1111-2222-3333-444455556666" (reference "C57") (unit 1)))))
+	(symbol (lib_id "power:+3V3") (at 58.42 199.39 0) (unit 1)
+		(exclude_from_sim no) (in_bom yes) (on_board yes) (dnp no)
+		(property "Reference" "#PWR430" (at 58.42 202.39 0) (effects (font (size 1.27 1.27)) (hide yes)))
+		(property "Value" "+3V3" (at 58.42 196.39 0) (effects (font (size 1.27 1.27))))
+		(instances (project "AUDIO_BOARD" (path "/ba93534c-f2e3-4dc0-9a76-585fdc68cf39/c0ffee00-1111-2222-3333-444455556666" (reference "#PWR430") (unit 1)))))
+	(wire (pts (xy 58.42 203.2) (xy 58.42 199.39)) (stroke (width 0) (type default)))
+	(symbol (lib_id "power:GND") (at 58.42 212.09 0) (unit 1)
+		(exclude_from_sim no) (in_bom yes) (on_board yes) (dnp no)
+		(property "Reference" "#PWR431" (at 58.42 215.09 0) (effects (font (size 1.27 1.27)) (hide yes)))
+		(property "Value" "GND" (at 58.42 209.09 0) (effects (font (size 1.27 1.27))))
+		(instances (project "AUDIO_BOARD" (path "/ba93534c-f2e3-4dc0-9a76-585fdc68cf39/c0ffee00-1111-2222-3333-444455556666" (reference "#PWR431") (unit 1)))))
+	(wire (pts (xy 58.42 208.28) (xy 58.42 212.09)) (stroke (width 0) (type default)))
 	(embedded_fonts no)
 )
