File: schematic/AUDIO_BOARD_v1_r1/routed_auto.kicad_pcb (KiCad board)
At the start: 4 copper layers, 101.5 x 79.9 mm, 167 parts, among them J1 PWR FFC 4p, J10 U.FL FX send R, J11 U.FL FX return L, J12 U.FL FX return R, J2 U.FL L in, J3 U.FL R in, J4 1/4in L, J5 1/4in R, J6 3.5mm HP, J7 CTRL FFC, J8 CTRL->PANEL FFC, J9 U.FL FX send L, Q1 MMBT3904, Q2 MMBT3906, Q3 MMBT3904, Q4 MMBT3906, U1 LTC660, U15 LTC660, U2 OPA1678, U20 DAC8565, U22 AP2112K-3.3, U3 OPA1678, U30 OPA1678, U31 LM13700, U32 LM13700, U33 4052, U34 OPA1678, U35 LM13700, U36 LM13700, U37 4052, U4 LM13700, U5 OPA1678, U6 4053, U7 DAC8565, U8 LM13700, U80 OPA1678

Commit message: try autorouter?
Routing:
- net /MASTER_FILTER/HPR: track 0.00 -> 84.2 mm, vias 0 -> 4
- net /VOL_R: track 0.00 -> 75.1 mm
- net Net-(U30B--): track 0.00 -> 73.3 mm, vias 0 -> 6
- net Net-(U30A--): track 0.00 -> 69.7 mm, vias 0 -> 9
- net /ANALOG_FILTER_CV/CV_VCA: track 0.00 -> 69.2 mm, vias 0 -> 5
- net /MF_MODE_A: track 0.00 -> 68.9 mm, vias 0 -> 4
- net /MF_CV_CUTOFF: track 0.00 -> 62.9 mm, vias 0 -> 7
- net Net-(U34A--): track 0.00 -> 62.5 mm, vias 0 -> 10
- net /MASTER_FILTER/HPL: track 0.00 -> 62.1 mm, vias 0 -> 8
- net /FILT_L_IN: track 0.00 -> 59.1 mm, vias 0 -> 4
- net /MF_CV_RES: track 0.00 -> 59.1 mm, vias 0 -> 5
- net /MF_MODE_B: track 0.00 -> 59.1 mm, vias 0 -> 6
- net /FILT_L_OUT: track 0.00 -> 56.1 mm, vias 0 -> 4
- net /MASTER_FILTER/BPL: track 0.00 -> 55.6 mm, vias 0 -> 7
- net /FX_RET_R: track 0.00 -> 54.4 mm, vias 0 -> 2
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