File: boards/AUDIO_BOARD/v1_r1/ANALOG_FILTER_CV.kicad_sch (KiCad schematic)
At the start: 30 parts, among them U4 LM13700, U5 OPA1678, U6 4053, U7 DAC8565, U8 LM13700

Commit message: rerouting
Connections:
- net FILT_L_IN: now also R30.2; no longer R30.1
- net at U4.3 (+): now also R30.1; no longer R30.2
Other:
- moved on the sheet: C90, R30
Changed lines of the file:
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@@
 	(wire
 		(pts
-			(xy 139.7 66.04) (xy 139.7 69.85)
+			(xy 203.708 229.362) (xy 203.708 233.172)
 		)
 		(stroke
@@
 	(wire
 		(pts
-			(xy 139.7 60.96) (xy 139.7 57.15)
+			(xy 203.708 224.282) (xy 203.708 220.472)
 		)
 		(stroke
@@
 	(symbol
 		(lib_id "Device:C_Small")
-		(at 139.7 63.5 0)
+		(at 203.708 226.822 0)
 		(unit 1)
 		(body_style 1)
@@
 		(fields_autoplaced yes)
 		(property "Reference" "C90"
-			(at 142.24 62.2362 0)
+			(at 206.248 225.5582 0)
 			(show_name no)
 			(do_not_autoplace no)
@@
 		)
 		(property "Value" "100nF"
-			(at 142.24 64.7762 0)
+			(at 206.248 228.0982 0)
 			(show_name no)
 			(do_not_autoplace no)
@@
 		)
 		(property "Footprint" "Capacitor_SMD:C_0402_1005Metric"
-			(at 139.7 63.5 0)
+			(at 203.708 226.822 0)
 			(hide yes)
 			(show_name no)
@@
 		)
 		(property "Datasheet" ""
-			(at 139.7 63.5 0)
+			(at 203.708 226.822 0)
 			(show_name no)
 			(do_not_autoplace no)
@@
 		)
 		(property "Description" ""
-			(at 139.7 63.5 0)
+			(at 203.708 226.822 0)
 			(show_name no)
 			(do_not_autoplace no)
@@
 	(symbol
 		(lib_id "power:GND")
-		(at 139.7 69.85 0)
+		(at 203.708 233.172 0)
 		(unit 1)
 		(body_style 1)
@@
 		(fields_autoplaced yes)
 		(property "Reference" "#PWR4059"
-			(at 139.7 72.39 0)
+			(at 203.708 235.712 0)
 			(hide yes)
 			(show_name no)
@@
 		)
 		(property "Value" "GND"
-			(at 142.24 71.1199 0)
+			(at 206.248 234.4419 0)
 			(show_name no)
 			(do_not_autoplace no)
@@
 		)
 		(property "Footprint" ""
-			(at 139.7 69.85 0)
+			(at 203.708 233.172 0)
 			(show_name no)
 			(do_not_autoplace no)
@@
 		)
 		(property "Datasheet" ""
-			(at 139.7 69.85 0)
+			(at 203.708 233.172 0)
 			(show_name no)
 			(do_not_autoplace no)
@@
 		)
 		(property "Description" ""
-			(at 139.7 69.85 0)
+			(at 203.708 233.172 0)
 			(show_name no)
 			(do_not_autoplace no)
@@
 	(symbol
 		(lib_id "Device:R")
-		(at 124.46 177.8 90)
+		(at 124.46 177.8 270)
+		(mirror x)
 		(unit 1)
 		(body_style 1)
@@
 		(in_pos_files yes)
 		(dnp no)
-		(fields_autoplaced yes)
 		(property "Reference" "R30"
 			(at 124.46 171.45 90)
@@
 	(symbol
 		(lib_id "power:+5V")
-		(at 139.7 57.15 0)
+		(at 203.708 220.472 0)
 		(unit 1)
 		(body_style 1)
@@
 		(fields_autoplaced yes)
 		(property "Reference" "#PWR4080"
-			(at 139.7 59.69 0)
+			(at 203.708 223.012 0)
 			(hide yes)
 			(show_name no)
@@
 		)
 		(property "Value" "+5V"
-			(at 142.24 55.8799 0)
+			(at 206.248 219.2019 0)
 			(show_name no)
 			(do_not_autoplace no)
@@
 		)
 		(property "Footprint" ""
-			(at 139.7 57.15 0)
+			(at 203.708 220.472 0)
 			(show_name no)
 			(do_not_autoplace no)
@@
 		)
 		(property "Datasheet" ""
-			(at 139.7 57.15 0)
+			(at 203.708 220.472 0)
 			(show_name no)
 			(do_not_autoplace no)
@@
 		)
 		(property "Description" ""
-			(at 139.7 57.15 0)
+			(at 203.708 220.472 0)
 			(show_name no)
 			(do_not_autoplace no)
