File: boards/AUDIO_BOARD/v1_r1/AUDIO_BOARD.kicad_sch (KiCad schematic)
At the start: 15 parts, among them J10 U.FL FX send R, J11 U.FL FX return L, J12 U.FL FX return R, J4 1/4in L, J5 1/4in R, J6 3.5mm HP, J7 CTRL FFC, J8 CTRL->PANEL FFC, J9 U.FL FX send L

Commit message: rerouting
Changed lines of the file:
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@@
 	(wire
 		(pts
-			(xy 242.57 68.58) (xy 250.11 68.83)
+			(xy 242.57 68.58) (xy 250.19 68.58)
 		)
 		(stroke
@@
 	(wire
 		(pts
-			(xy 250.19 59.69) (xy 249.97 67.96)
-		)
-		(stroke
-			(width 0)
-			(type default)
-		)
-	)
-	(wire
-		(pts
 			(xy 347.98 63.5) (xy 355.6 63.5)
 		)
@@
 	)
 	(label "FILT_R_IN"
-		(at 250.11 68.83 0)
+		(at 250.19 68.58 0)
 		(effects
 			(font
@@
 	(symbol
 		(lib_id "power:PWR_FLAG")
-		(at 245.11 68.58 0)
+		(at 272.288 69.85 0)
 		(unit 1)
 		(body_style 1)
@@
 		(fields_autoplaced yes)
 		(property "Reference" "#FLG9002"
-			(at 237.49 71.12 0)
+			(at 264.668 72.39 0)
 			(hide yes)
 			(show_name no)
@@
 		)
 		(property "Value" "PWR_FLAG"
-			(at 247.65 67.3099 0)
+			(at 274.32 68.5799 0)
 			(show_name no)
 			(do_not_autoplace no)
@@
 		)
 		(property "Footprint" ""
-			(at 237.49 68.58 0)
+			(at 264.668 69.85 0)
 			(show_name no)
 			(do_not_autoplace no)
@@
 		)
 		(property "Datasheet" ""
-			(at 237.49 68.58 0)
+			(at 264.668 69.85 0)
 			(show_name no)
 			(do_not_autoplace no)
@@
 		)
 		(property "Description" ""
-			(at 237.49 68.58 0)
+			(at 264.668 69.85 0)
 			(show_name no)
 			(do_not_autoplace no)
@@
 				(path "/f48c9b16-466a-451c-a18e-f0696896ad19"
 					(reference "#FLG9002")
-					(unit 1)
-				)
-			)
-		)
-	)
-	(symbol
-		(lib_id "power:GND")
-		(at 249.97 67.96 0)
-		(unit 1)
-		(body_style 1)
-		(exclude_from_sim no)
-		(in_bom yes)
-		(on_board yes)
-		(in_pos_files yes)
-		(dnp no)
-		(fields_autoplaced yes)
-		(property "Reference" "#PWR4005"
-			(at 250.19 71.12 0)
-			(hide yes)
-			(show_name no)
-			(do_not_autoplace no)
-			(effects
-				(font
-					(size 1.27 1.27)
-				)
-			)
-		)
-		(property "Value" "GND"
-			(at 252.73 69.2299 0)
-			(show_name no)
-			(do_not_autoplace no)
-			(effects
-				(font
-					(size 1.27 1.27)
-				)
-				(justify left)
-			)
-		)
-		(property "Footprint" ""
-			(at 249.97 67.96 0)
-			(show_name no)
-			(do_not_autoplace no)
-			(effects
-				(font
-					(size 1.27 1.27)
-				)
-			)
-		)
-		(property "Datasheet" ""
-			(at 249.97 67.96 0)
-			(show_name no)
-			(do_not_autoplace no)
-			(effects
-				(font
-					(size 1.27 1.27)
-				)
-			)
-		)
-		(property "Description" ""
-			(at 249.97 67.96 0)
-			(show_name no)
-			(do_not_autoplace no)
-			(effects
-				(font
-					(size 1.27 1.27)
-				)
-			)
-		)
-		(pin "1"
-		)
-		(instances
-			(project "AUDIO_BOARD"
-				(path "/f48c9b16-466a-451c-a18e-f0696896ad19"
-					(reference "#PWR4005")
 					(unit 1)
 				)
@@
 	(symbol
 		(lib_id "power:GND")
-		(at 245.11 68.58 0)
+		(at 272.288 69.85 0)
 		(unit 1)
 		(body_style 1)
@@
 		(fields_autoplaced yes)
 		(property "Reference" "#PWR9002"
-			(at 250.19 71.12 0)
+			(at 277.368 72.39 0)
 			(hide yes)
 			(show_name no)
@@
 		)
 		(property "Value" "GND"
-			(at 247.65 69.8499 0)
+			(at 274.32 71.1199 0)
 			(show_name no)
 			(do_not_autoplace no)
@@
 		)
 		(property "Footprint" ""
-			(at 249.97 67.96 0)
+			(at 277.148 69.23 0)
 			(show_name no)
 			(do_not_autoplace no)
@@
 		)
 		(property "Datasheet" ""
-			(at 249.97 67.96 0)
+			(at 277.148 69.23 0)
 			(show_name no)
 			(do_not_autoplace no)
@@
 		)
 		(property "Description" ""
-			(at 249.97 67.96 0)
+			(at 277.148 69.23 0)
 			(show_name no)
 			(do_not_autoplace no)
@@
 	(symbol
 		(lib_id "power:PWR_FLAG")
-		(at 252.73 68.58 180)
+		(at 272.288 63.5 180)
 		(unit 1)
 		(body_style 1)
@@
 		(fields_autoplaced yes)
 		(property "Reference" "#FLG9010"
-			(at 237.49 71.12 0)
+			(at 257.048 66.04 0)
 			(hide yes)
 			(show_name no)
@@
 		)
 		(property "Value" "PWR_FLAG"
-			(at 255.27 69.8499 0)
+			(at 274.32 64.7699 0)
 			(show_name no)
 			(do_not_autoplace no)
@@
 		)
 		(property "Footprint" ""
-			(at 237.49 68.58 0)
+			(at 257.048 63.5 0)
 			(show_name no)
 			(do_not_autoplace no)
@@
 		)
 		(property "Datasheet" ""
-			(at 237.49 68.58 0)
+			(at 257.048 63.5 0)
 			(show_name no)
 			(do_not_autoplace no)
@@
 		)
 		(property "Description" ""
-			(at 237.49 68.58 0)
+			(at 257.048 63.5 0)
 			(show_name no)
 			(do_not_autoplace no)
@@
 	(symbol
 		(lib_id "power:+5V")
-		(at 252.73 68.58 0)
+		(at 272.288 63.5 0)
 		(unit 1)
 		(body_style 1)
@@
 		(fields_autoplaced yes)
 		(property "Reference" "#PWR9010"
-			(at 250.19 71.12 0)
+			(at 269.748 66.04 0)
 			(hide yes)
 			(show_name no)
@@
 		)
 		(property "Value" "+5V"
-			(at 255.27 67.3099 0)
+			(at 274.32 62.2299 0)
 			(show_name no)
 			(do_not_autoplace no)
@@
 		)
 		(property "Footprint" ""
-			(at 249.97 67.96 0)
+			(at 269.528 62.88 0)
 			(show_name no)
 			(do_not_autoplace no)
@@
 		)
 		(property "Datasheet" ""
-			(at 249.97 67.96 0)
+			(at 269.528 62.88 0)
 			(show_name no)
 			(do_not_autoplace no)
@@
 		)
 		(property "Description" ""
-			(at 249.97 67.96 0)
+			(at 269.528 62.88 0)
 			(show_name no)
 			(do_not_autoplace no)
@@
 		(fields_autoplaced yes)
 		(property "Reference" "H3"
-			(at 110.49 304.7999 0)
-			(show_name no)
-			(do_not_autoplace no)
-			(effects
-				(font
-					(size 1.27 1.27)
-				)
-				(justify left)
+			(at 107.95 299.72 0)
+			(show_name no)
+			(do_not_autoplace no)
+			(effects
+				(font
+					(size 1.27 1.27)
+				)
 			)
 		)
 		(property "Value" "M2"
-			(at 110.49 307.3399 0)
-			(show_name no)
-			(do_not_autoplace no)
-			(effects
-				(font
-					(size 1.27 1.27)
-				)
-				(justify left)
-			)
-		)
+			(at 107.95 302.26 0)
+			(show_name no)
+			(do_not_autoplace no)
+			(effects
+				(font
+					(size 1.27 1.27)
+				)
+			)
+		)
