File: boards/FILTER_BOARD/v1_r1/FILTER.kicad_sch (KiCad schematic)
At the start: 71 parts, among them J13 U.FL AUDIO L IN, J14 U.FL AUDIO R IN, J15 U.FL AUDIO L OUT, J16 U.FL AUDIO R OUT, J17 FILTER FFC, U30 OPA1678, U31 LM13700, U32 LM13700, U33 4052, U34 OPA1678, U35 LM13700, U36 LM13700, U37 4052

Commit message: trying panelization?
Parts:
- removed J13: U.FL AUDIO L IN, Connector_Coaxial:U.FL_Hirose_U.FL-R-SMT-1_Vertical, symbol Connector:Conn_Coaxial_Small
- removed J14: U.FL AUDIO R IN, Connector_Coaxial:U.FL_Hirose_U.FL-R-SMT-1_Vertical, symbol Connector:Conn_Coaxial_Small
- removed J15: U.FL AUDIO L OUT, Connector_Coaxial:U.FL_Hirose_U.FL-R-SMT-1_Vertical, symbol Connector:Conn_Coaxial_Small
- removed J16: U.FL AUDIO R OUT, Connector_Coaxial:U.FL_Hirose_U.FL-R-SMT-1_Vertical, symbol Connector:Conn_Coaxial_Small
- removed J17: FILTER FFC, Connector_FFC-FPC:Hirose_FH12-10S-0.5SH_1x10-1MP_P0.50mm_Horizontal, symbol Connector_Generic:Conn_01x10
- added J1: U.FL AUDIO L IN, Connector_Coaxial:U.FL_Hirose_U.FL-R-SMT-1_Vertical, symbol Connector:Conn_Coaxial_Small
- added J2: U.FL AUDIO R IN, Connector_Coaxial:U.FL_Hirose_U.FL-R-SMT-1_Vertical, symbol Connector:Conn_Coaxial_Small
- added J3: U.FL AUDIO L OUT, Connector_Coaxial:U.FL_Hirose_U.FL-R-SMT-1_Vertical, symbol Connector:Conn_Coaxial_Small
- added J4: U.FL AUDIO R OUT, Connector_Coaxial:U.FL_Hirose_U.FL-R-SMT-1_Vertical, symbol Connector:Conn_Coaxial_Small
- added J5: FILTER FFC, Connector_FFC-FPC:Hirose_FH12-10S-0.5SH_1x10-1MP_P0.50mm_Horizontal, symbol Connector_Generic:Conn_01x10
Connections:
- net AUDIO_L_IN: now also J1.1 (In)
- net AUDIO_L_OUT: now also J3.1 (In)
- net AUDIO_R_IN: now also J2.1 (In)
- net AUDIO_R_OUT: now also J4.1 (In)
- net CV_CUTOFF: now also J5.4 (Pin_4)
- net CV_RES: now also J5.6 (Pin_6)
- net MODE_A: now also J5.8 (Pin_8)
- net MODE_B: now also J5.9 (Pin_9)
- net FILT_+5V renamed +5V
- net +5V: now also J5.1 (Pin_1)
- net FILT_-5V renamed -5V
- net -5V: now also J5.2 (Pin_2)
- net FILT_GND renamed GND
- net GND: now also J1.2 (Ext), J2.2 (Ext), J3.2 (Ext), J4.2 (Ext), J5.10 (Pin_10), J5.3 (Pin_3), J5.5 (Pin_5), J5.7 (Pin_7)
