File: boards/APM/v6_r1/APM.kicad_pcb (KiCad board)
At the start: 4 copper layers, 72.5 x 111.9 mm, 131 parts, among them J1 DF40C-60DS-0.4V(51), J11 DAC_L_PRB, J12 Conn_01x02, J16 USB_A_FEMALE, J19 AudioPlug3, J2 AUDIO_PWR, J23 VOL_L_CTRL, J24 VOL_R_CTRL, J3 DF40C-60DS-0.4V(51), J30 UART_DEBUG, J31 Conn_02x04_Odd_Even, J4 LCD_display, J5 Barrel_Jack, J6 OSC_CTRL, J7 DAC_R_PRB, J8 AUDIO_CTRL, SW1 RST, U13 INA219AxD, U2 OPA1678, U3 LT1963AxST-3.3, U4 W25Q128JVS, U5 MR25H40, U6 W25Q128JVS, U7 INA219AxD, U8 24LC1025-I_P, U9 USBLC6-2SC6

Commit message: such a pain, still trying to get it routed
Parts:
- moved C17 59.0 mm to (71.5, 146.3), turned to 180 degrees
- moved L5 6.46 mm to (115.7, 146.3)
- moved R98 6.46 mm to (115.7, 144.5)
- moved SW1 6.46 mm to (119.6, 145.7)
- moved C24 6.42 mm to (114.3, 146.3), turned to 90 degrees
- moved R96 1.31 mm to (111.4, 142.6)
- moved R97 1.31 mm to (111.4, 141.7)
Routing:
- net /FPGA_INTERFACE/D7_DONE: track 0.00 -> 31.3 mm, vias 0 -> 3
- net /FPGA_INTERFACE/H11_IOT3A_S1: track 0.00 -> 23.8 mm, vias 0 -> 2
- net /FPGA_INTERFACE/E8_READY: track 0.00 -> 19.1 mm, vias 0 -> 1
- net /FPGA_INTERFACE/FPGA_3V3: track 16.3 -> 33.1 mm
- net /FPGA_INTERFACE/RST_NODE: track 0.00 -> 5.74 mm
- net 5V_APM: track 226.4 -> 228.2 mm
- net FPGA_5V: track 12.1 -> 11.2 mm

Commit message: routed, dfc connector mixup?
Parts:
- added C25: 220uF 10V, Capacitor_SMD:CP_Elec_4x3, B.Cu at (124.3, 56.7)
- moved J2 2.06 mm to (129.6, 56.2)
Routing:
- net /FPGA_INTERFACE/A2_JTAG_TDO: track 0.00 -> 42.1 mm, vias 0 -> 2
- net /FPGA_INTERFACE/B1_JTAG_TMS: track 0.00 -> 38.9 mm, vias 0 -> 3
- net /FPGA_INTERFACE/FPGA_3V3: track 33.1 -> 70.2 mm, vias 2 -> 6
- net /APM_FPGA_UART_RX: track 58.9 -> 92.8 mm, vias 2 -> 5
- net /APM_FPGA_UART_TX: track 49.6 -> 82.6 mm, vias 2 -> 4
- net /FPGA_INTERFACE/A3_JTAG_TDI: track 0.00 -> 32.5 mm, vias 0 -> 3
- net /FPGA_INTERFACE/E8_READY: track 19.1 -> 48.3 mm, vias 1 -> 5
- net /FPGA_INTERFACE/C1_JTAG_TCK: track 11.4 -> 37.1 mm, vias 0 -> 3
- net /FPGA_INTERFACE/VCCIO23: track 1.94 -> 26.3 mm, vias 0 -> 2
- net /FPGA_INTERFACE/VCCIO01: track 1.94 -> 22.9 mm, vias 0 -> 2
- net /FPGA_INTERFACE/VCCIO67: track 1.94 -> 22.2 mm, vias 0 -> 2
- net /FPGA_INTERFACE/D7_DONE: track 31.3 -> 42.1 mm, vias 3 -> 4
- net 5V_APM: track 228.2 -> 235.8 mm, vias 13 -> 11
- net GND: track 2.15 -> 6.62 mm, vias 24 -> 30
Other:
- board text removed: "ACB_PWR"

Commit message: ready for fab??
Other:
- board text added: "3v3"
- board text added: "RX"
- board text added: "TCK"
- board text added: "TDI"
- board text added: "TDO"
- board text added: "TMS"
- board text added: "TX"
Changed lines of the file:
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@@
 		)
 		(embedded_fonts no)
-		(model "/home/akiel/trunk/pub/my_footprints/DF40C-60DP-0.4V_51_.step"
+		(model "/home/akiel/trunk/pub/my_footprints/DF40C-60DP.stp"
 			(offset
-				(xyz -6.76 -0.15 0.6)
+				(xyz -6.77 0 0.65)
 			)
 			(scale
@@
 		(layer "B.SilkS")
 		(effects
+			(font
+				(size 0.4 0.4)
+				(thickness 0.05)
+			)
+			(justify mirror)
+		)
+	)
+	(gr_text "TDI"
+		(at 113.49 133.9 0)
+		(layer "B.SilkS")
+		(effects
+			(font
+				(size 0.4 0.4)
+				(thickness 0.05)
+			)
+			(justify mirror)
+		)
+	)
+	(gr_text "3v3"
+		(at 113.49 136.47 0)
+		(layer "B.SilkS")
+		(effects
+			(font
+				(size 0.4 0.4)
+				(thickness 0.05)
+			)
+			(justify mirror)
+		)
+	)
+	(gr_text "GND"
+		(at 113.49 138.98 0)
+		(layer "B.SilkS")
+		(effects
+			(font
+				(size 0.4 0.4)
+				(thickness 0.05)
+			)
+			(justify mirror)
+		)
+	)
+	(gr_text "TX"
+		(at 113.49 141.52 0)
+		(layer "B.SilkS")
+		(effects
+			(font
+				(size 0.4 0.4)
+				(thickness 0.05)
+			)
+			(justify mirror)
+		)
+	)
+	(gr_text "TMS"
+		(at 123.61 133.9 0)
+		(layer "B.SilkS")
+		(effects
+			(font
+				(size 0.4 0.4)
+				(thickness 0.05)
+			)
+			(justify mirror)
+		)
+	)
+	(gr_text "TCK"
+		(at 123.61 136.44 0)
+		(layer "B.SilkS")
+		(effects
+			(font
+				(size 0.4 0.4)
+				(thickness 0.05)
+			)
+			(justify mirror)
+		)
+	)
+	(gr_text "TDO"
+		(at 123.61 139.05 0)
+		(layer "B.SilkS")
+		(effects
+			(font
+				(size 0.4 0.4)
+				(thickness 0.05)
+			)
+			(justify mirror)
+		)
+	)
+	(gr_text "RX"
+		(at 123.61 141.52 0)
+		(layer "B.SilkS")
+		(effects
