File: boards/APM/v6_r1_rert/APM.kicad_sch (KiCad schematic)
At the start: 25 parts, among them J2 AUDIO_PWR, J4 LCD_display, J6 OSC_CTRL, J8 AUDIO_CTRL

Commit message: new APM rerouted looks better, passes DRC...
Parts:
- removed 3v3: 3v3, TestPoint:TestPoint_Pad_D1.0mm, symbol Connector:TestPoint
- removed GND1: GND, TestPoint:TestPoint_Pad_D1.0mm, symbol Connector:TestPoint
- added C25: 220uF 10V, Capacitor_SMD:CP_Elec_4x3, symbol Device:C_Small
Connections:
- net 5V_APM: now also C25.1
- net GND: now also C25.2
