File: boards/APM/v6_r1_rert/FPGA_INTERFACE.kicad_sch (KiCad schematic)
At the start: 35 parts, among them J1 DF40C-60DS-0.4V(51), J15 FPGA FFC, J21 FPGA FMC, J3 DF40C-60DS-0.4V(51), J31 Conn_02x04_Odd_Even, SW1 RST

Commit message: new APM rerouted looks better, passes DRC...
Parts:
- removed TP10, TP11, TP12, TP13, TP14: TestPoint, TestPoint:TestPoint_Pad_D1.0mm, symbol Connector:TestPoint
- J1, J3: footprint my_footprints:HIROSE_DF40C-60DP-0.4V_51_ -> my_footprints:Hirose_DF40C-60DS-0.4V_2x30_P0.4mm
Connections:
- net D7_DONE: now also J1.25 (Pin_25)
- net E8_READY: now also J1.17 (Pin_17)
- net FPGA_3V3: now also J3.48 (Pin_48), J3.50 (Pin_50)
- net FPGA_5V: now also J3.52 (Pin_52), J3.54 (Pin_54), J3.56 (Pin_56), J3.58 (Pin_58)
- net H11_IOT3A_S1: now also J1.3 (Pin_3)
- net VCCIO01: now also J1.24 (Pin_24), J1.26 (Pin_26)
- net VCCIO23: now also J3.2 (Pin_2), J3.4 (Pin_4)
- net VCCIO67: now also J1.29 (Pin_29), J1.31 (Pin_31)
