File: boards/APM/v7_r1/APM.kicad_sch (KiCad schematic)
At the start: 24 parts, among them J2 AUDIO_PWR, J4 LCD_display, J6 OSC_CTRL, J8 AUDIO_CTRL

Commit message: more placement
Connections:
- net DAC_1-1_R: no longer U1.32 (PA4)
- net DAC_1-2_L: no longer U10.11 (PA5)
- new net DAC_1-1_L: U1.32 (PA4)
- new net DAC_1-2_R: U10.11 (PA5)
Changed lines of the file:
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@@
 		)
 	)
-	(label "DAC_1-2_L"
+	(label "DAC_1-2_R"
 		(at 236.22 39.37 180)
 		(effects
@@
 		)
 	)
-	(label "DAC_1-1_R"
+	(label "DAC_1-1_L"
 		(at 298.45 62.23 0)
 		(effects
