File: boards/APM/v7_r1/APM.kicad_pcb (KiCad board)
At the start: 6 copper layers, 72.5 x 111.9 mm, 154 parts, among them J1 DF40C-60DS-0.4V(51), J11 DAC_L_PRB, J13 ACM_DAC_L, J16 USB_A_FEMALE, J2 AUDIO_PWR, J3 DF40C-60DS-0.4V(51), J30 UART_DEBUG, J31 Conn_02x04_Odd_Even, J4 LCD_display, J5 Barrel_Jack, J6 OSC_CTRL, J7 DAC_R_PRB, J8 AUDIO_CTRL, J9 ACM_DAC_R, SW1 RST, U11 CS4344, U12 OPA1656ID, U13 INA219AxD, U14 LTC660, U3 LT1963AxST-3.3, U4 W25Q128JVS, U5 MR25H40, U6 W25Q128JVS, U7 INA219AxD, U8 24LC1025-I_P, U9 USBLC6-2SC6

Commit message: autorouting
Parts:
- moved F2 6.58 mm to (74.0, 136.4)
- moved C19 6.58 mm to (74.0, 129.7)
- moved D64 6.58 mm to (74.0, 134.3)
Routing:
- net 5V_APM: track 40.6 -> 193.2 mm, vias 1 -> 19
- net /FPGA_INTERFACE/FPGA_3V3: track 1.57 -> 135.1 mm, vias 0 -> 9
- net /APM_FMC_NWAIT: track 0.00 -> 113.8 mm, vias 0 -> 1
- net /APM_I2C2_SDA: track 2.25 -> 112.9 mm, vias 0 -> 6
- net /APM_I2C2_SCL: track 2.26 -> 111.7 mm, vias 0 -> 4
- net /APM_FMC_DA13: track 0.00 -> 102.3 mm, vias 0 -> 1
- net /APM_FPGA_UART_RX: track 0.00 -> 95.5 mm, vias 0 -> 3
- net /APM_SPI1_SCK: track 0.00 -> 88.9 mm, vias 0 -> 5
- net /QSPI1_NCS: track 0.00 -> 87.0 mm, vias 0 -> 1
- net /APM_FPGA_UART_TX: track 0.00 -> 85.0 mm, vias 0 -> 4
- net /APM_SPI1_MISO: track 0.00 -> 84.8 mm, vias 0 -> 5
- net /AUD_GATE: track 0.00 -> 82.5 mm, vias 0 -> 3
- net /AUD_SPARE: track 0.00 -> 78.8 mm, vias 0 -> 2
- net /AUD_CS_POTS: track 0.00 -> 72.6 mm, vias 0 -> 2
- net /QSPI_SCK2: track 0.00 -> 67.4 mm, vias 0 -> 1
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- added copper zone on In3.Cu, net 3V3_APM
- added copper zone on In1.Cu, net GND
- removed copper zone on In1.Cu, net 3V3_APM
- removed copper zone on In2.Cu, net GND
- removed copper zone on In3.Cu, net GND

Commit message: autorouting. more of it
Routing:
- net 5V_APM: track 193.2 -> 62.4 mm, vias 19 -> 30
- net 3V3_APM: track 38.3 -> 76.9 mm, vias 13 -> 16
- net FPGA_5V: track 23.6 -> 0.00 mm, vias 2 -> 7
- net GND: vias 30 -> 462
- net /FPGA_INTERFACE/FPGA_3V3: vias 9 -> 13
- added copper zone on In3.Cu, net /FPGA_INTERFACE/FPGA_3V3
- added copper zone on In3.Cu, net 5V_APM
- added copper zone on In3.Cu, net FPGA_5V
